File: hardware/v2/artix7-pcie-v2-bank14.sch (KiCad schematic (older format))
At the start: 5 parts, among them J2 Conn_02x20_Odd_Even, U1 XC7A75T-FGG484

Commit message: v2 pcb/schematic update : drc passing, need to add caps
Connections:
- net IO_L21_14_P: now reaches U1.N17 (IO_L21P_T3_DQS_14)
- net IO_L21_14_N: now reaches U1.P17 (IO_L21N_T3_DQS_A06_D22_14)
- net IO_L22_14_N: now reaches U1.R16 (IO_L22N_T3_A04_D20_14)
- net IO_L24_14_N: now reaches U1.R17 (IO_L24N_T3_A00_D16_14)
- net IO_L13_14_N: now reaches U1.Y19 (IO_L13N_T2_MRCC_14)
- net +3V3 renamed VCCO_14
- net VCCO_14: no longer J2.19 (Pin_19), J2.20 (Pin_20), J2.39 (Pin_39), J2.40 (Pin_40)
- new net VCCO_16: J2.19 (Pin_19), J2.20 (Pin_20), J2.39 (Pin_39), J2.40 (Pin_40)
- no-connect marks 48 -> 42
Changed lines of the file:
@@
 EESchema Schematic File Version 4
-LIBS:artix7-pcie-v2-cache
 EELAYER 30 0
 EELAYER END
 $Descr A4 11693 8268
 encoding utf-8
-Sheet 6 7
+Sheet 4 7
 Title ""
 Date ""
@@
 Wire Wire Line
 	5150 2800 5500 2800
-Wire Wire Line
-	1550 700  1550 900
-Wire Wire Line
-	4750 900  4750 700
 $Comp
 L tom-passives:R R8
@@
 	1    0    0    1
 $EndComp
-Wire Wire Line
-	9300 5900 8450 5900
-Wire Wire Line
-	9800 5900 10800 5900
-Wire Wire Line
-	9300 5000 8450 5000
-Wire Wire Line
-	8450 5000 8450 5900
-Wire Wire Line
-	10800 5000 10800 5900
-Wire Wire Line
-	9300 4000 8450 4000
-Wire Wire Line
-	8450 4000 8450 5000
-Connection ~ 8450 5000
-Wire Wire Line
-	9800 4000 10800 4000
-Wire Wire Line
-	10800 4000 10800 5000
-Connection ~ 10800 5000
 Wire Wire Line
 	8550 4100 9300 4100
@@
 Text HLabel 9150 4200 0    50   BiDi ~ 0
 IO_L9_16_N
-$Comp
-L power:+3V3 #PWR0105
-U 1 1 5ED5D308
-P 10800 4000
-F 0 "#PWR0105" H 10800 3850 50  0001 C CNN
-F 1 "+3V3" H 10815 4173 50  0000 C CNN
-F 2 "" H 10800 4000 50  0001 C CNN
-F 3 "" H 10800 4000 50  0001 C CNN
-	1    10800 4000
-	1    0    0    -1
-$EndComp
-Connection ~ 10800 4000
-$Comp
-L power:+3V3 #PWR0106
-U 1 1 5ED5F3A8
-P 8450 4000
-F 0 "#PWR0106" H 8450 3850 50  0001 C CNN
-F 1 "+3V3" H 8465 4173 50  0000 C CNN
-F 2 "" H 8450 4000 50  0001 C CNN
-F 3 "" H 8450 4000 50  0001 C CNN
-	1    8450 4000
-	1    0    0    -1
-$EndComp
-Connection ~ 8450 4000
 Wire Wire Line
 	9800 4200 9950 4200
@@
 IO_L4_14_P
 Wire Wire Line
-	9800 5000 10800 5000
-Wire Wire Line
 	9950 5100 9800 5100
 Wire Wire Line
@@
 Wire Wire Line
 	5300 3300 5150 3300
-$Comp
-L power:+3V3 #PWR0120
-U 1 1 5F093C5F
-P 4750 700
-F 0 "#PWR0120" H 4750 550 50  0001 C CNN
-F 1 "+3V3" H 4765 873 50  0000 C CNN
-F 2 "" H 4750 700 50  0001 C CNN
-F 3 "" H 4750 700 50  0001 C CNN
-	1    4750 700
-	1    0    0    -1
-$EndComp
 NoConn ~ 5150 1700
 NoConn ~ 5150 2600
@@
 NoConn ~ 5150 2900
 NoConn ~ 5150 3800
-NoConn ~ 5150 4300
 NoConn ~ 5150 5500
 NoConn ~ 5150 5600
-NoConn ~ 5150 5800
-NoConn ~ 5150 5900
-NoConn ~ 5150 6100
-NoConn ~ 5150 6500
 NoConn ~ 1150 1700
 NoConn ~ 1150 2200
@@
 NoConn ~ 1150 2000
 NoConn ~ 1150 2100
-Connection ~ 4750 900
 Wire Wire Line
 	1850 900  1950 900
@@
 	1550 900  1650 900
 Connection ~ 1650 900
-Connection ~ 1550 900
 $Comp
 L artix7-pcie-v2:XC7A75T-FGG484 U1
@@
 NoConn ~ 1150 2400
 NoConn ~ 1150 2500
-NoConn ~ 1550 700
-Text Label 1550 700  0    50   ~ 0
+Text Label 1950 900  0    50   ~ 0
 VCCO_13
 Text HLabel 5300 4000 2    50   Input ~ 0
@@
 Wire Wire Line
 	5150 5700 5300 5700
+Text HLabel 4950 900  2    50   Input ~ 0
+VCCO_14
+Wire Wire Line
+	4950 900  4750 900
+Connection ~ 4750 900
+Text HLabel 8350 3850 0    50   Input ~ 0
+VCCO_16
+Wire Wire Line
+	4250 900  3950 900
+Connection ~ 4250 900
+Text Label 3950 900  2    50   ~ 0
+VCCO_14
+Text Label 9150 5900 2    50   ~ 0
+VCCO_14
+Text Label 9950 5900 0    50   ~ 0
+VCCO_14
+Wire Wire Line
+	8450 5000 8450 4000
+Wire Wire Line
+	8450 5000 9300 5000
+Connection ~ 8450 3850
+Wire Wire Line
+	8450 3850 8350 3850
+Wire Wire Line
+	10800 3850 10800 4000
+Wire Wire Line
+	10800 5000 9800 5000
+Wire Wire Line
+	8450 3850 10800 3850
+Wire Wire Line
+	9300 4000 8450 4000
+Connection ~ 8450 4000
+Wire Wire Line
+	8450 4000 8450 3850
+Wire Wire Line
+	9800 4000 10800 4000
+Connection ~ 10800 4000
+Wire Wire Line
+	10800 4000 10800 5000
+Wire Wire Line
+	9150 5900 9300 5900
+Wire Wire Line
+	9800 5900 9950 5900
+Text HLabel 5300 4300 2    50   Input ~ 0
+IO_L13_14_N
+Wire Wire Line
+	5300 4300 5150 4300
+Text HLabel 5300 5900 2    50   BiDi ~ 0
+IO_L21_14_N
+Text HLabel 5300 5800 2    50   Output ~ 0
+IO_L21_14_P
+Wire Wire Line
+	5300 5800 5150 5800
+Wire Wire Line
+	5150 5900 5300 5900
+$Comp
+L power:PWR_FLAG #FLG0110
+U 1 1 5EE3E044
+P 1550 900
+F 0 "#FLG0110" H 1550 975 50  0001 C CNN
+F 1 "PWR_FLAG" H 1550 1073 50  0000 C CNN
+F 2 "" H 1550 900 50  0001 C CNN
+F 3 "~" H 1550 900 50  0001 C CNN
+	1    1550 900
+	1    0    0    -1
+$EndComp
+Connection ~ 1550 900
+Text HLabel 5300 6100 2    50   Input ~ 0
+IO_L22_14_N
+Wire Wire Line
+	5300 6100 5150 6100
+Text HLabel 5300 6500 2    50   Input ~ 0
+IO_L24_14_N
+Wire Wire Line
+	5300 6500 5150 6500
 $EndSCHEMATC

Commit message: v2 hardware: pcb progress commit, 155 unrouted
Parts:
- added C60, C67, C68: 100uF/6.3V/X5R, tom-passives:C_1206_3216Metric, symbol tom-passives:C
- added C61, C62: 4.7uF/6.3V/X5R, tom-passives:C_0402_1005Metric, symbol tom-passives:C
- added C63, C64, C65, C66: 0.47uF/6.3V/X5R, tom-passives:C_0402_1005Metric, symbol tom-passives:C
Connections:
- net GND: now also C60.2, C61.2, C62.2, C63.2, C64.2, C65.2, C66.2, C67.2, C68.2
- net VCCO_14: now also C60.1, C61.1, C62.1, C63.1, C64.1, C65.1, C66.1, C67.1
- net VCCO_16: now also C68.1
- net IO_L5_14_P: now reaches U1.P19 (IO_L5P_T0_D06_14)
- net IO_L0_14: now reaches U1.P20 (IO_0_14)
- net IO_L5_14_N: now reaches U1.R19 (IO_L5N_T0_D07_14)
- net IO_L11_14_P: now reaches U1.U20 (IO_L11P_T1_SRCC_14)
- net PUDC_14: now reaches R8.2, U1.U22 (IO_L3P_T0_DQS_PUDC_B_14)
- net IO_L20_14_N: no longer names the net of U1.T18 (IO_L20N_T3_A07_D23_14)
- net IO_L23_14_N: no longer names the net of U1.N14 (IO_L23N_T3_A02_D18_14)
- net IO_L23_14_P: no longer names the net of U1.N13 (IO_L23P_T3_A03_D19_14)
- net IO_L25_14: no longer names the net of U1.N15 (IO_25_14)
- no-connect marks 42 -> 41
Other:
- note added: "ULX3S"

Commit message: v2 pcb/schematic progress commit, all tough signals routed out
Connections:
- net IO_L9_16_N is gone; now on net IO_L11_16_N: J2.35 (Pin_35)
- net IO_L9_16_P is gone; now on net IO_L11_16_P: J2.36 (Pin_36)
- net IO_L11_16_N: no longer J2.33 (Pin_33)
- net IO_L11_16_P: no longer J2.34 (Pin_34)
- net IO_L17_16_N: now also J2.33 (Pin_33); no longer J2.31 (Pin_31)
- net IO_L17_16_P: now also J2.34 (Pin_34); no longer J2.32 (Pin_32)
- net IO_L20_16_N: now also J2.29 (Pin_29); no longer J2.27 (Pin_27)
- net IO_L20_16_P: now also J2.30 (Pin_30); no longer J2.28 (Pin_28)
- net IO_L21_16_N: now also J2.31 (Pin_31); no longer J2.29 (Pin_29)
- net IO_L21_16_P: now also J2.32 (Pin_32); no longer J2.30 (Pin_30)
- net IO_L22_16_N: now also J2.27 (Pin_27); no longer J2.25 (Pin_25)
- net IO_L22_16_P: now also J2.28 (Pin_28); no longer J2.26 (Pin_26)
- new net IO_L23_16_N: J2.25 (Pin_25)
- new net IO_L23_16_P: J2.26 (Pin_26)
Changed lines of the file:
@@
 	8550 4100 9300 4100
 Wire Wire Line
-	8550 4100 8550 4900
-Wire Wire Line
-	8550 4900 9300 4900
-Wire Wire Line
-	8550 4900 8550 5800
-Wire Wire Line
 	8550 5800 9300 5800
-Connection ~ 8550 4900
 Wire Wire Line
 	9800 4100 10700 4100
@@
 EndData
 $EndBitmap
-Text HLabel 9950 4200 2    50   BiDi ~ 0
-IO_L9_16_P
-Text HLabel 9150 4200 0    50   BiDi ~ 0
-IO_L9_16_N
-Wire Wire Line
-	9800 4200 9950 4200
-Wire Wire Line
-	9300 4200 9150 4200
 $Comp
 L power:GND #PWR025
@@
 	8550 5800 8550 6000
 Connection ~ 8550 5800
+Text HLabel 9950 4300 2    50   BiDi ~ 0
+IO_L17_16_P
+Text HLabel 9150 4300 0    50   BiDi ~ 0
+IO_L17_16_N
+Text HLabel 9150 4400 0    50   BiDi ~ 0
+IO_L21_16_N
 Text HLabel 9950 4400 2    50   BiDi ~ 0
-IO_L17_16_P
-Text HLabel 9150 4400 0    50   BiDi ~ 0
-IO_L17_16_N
+IO_L21_16_P
+Text HLabel 9950 4500 2    50   BiDi ~ 0
+IO_L20_16_P
 Text HLabel 9150 4500 0    50   BiDi ~ 0
-IO_L21_16_N
-Text HLabel 9950 4500 2    50   BiDi ~ 0
-IO_L21_16_P
-Text HLabel 9950 4600 2    50   BiDi ~ 0
-IO_L20_16_P
-Text HLabel 9150 4600 0    50   BiDi ~ 0
 IO_L20_16_N
 Text HLabel 9150 4800 0    50   BiDi ~ 0
@@
 Text HLabel 9950 4800 2    50   BiDi ~ 0
 IO_L24_16_P
-Text HLabel 9150 4300 0    50   BiDi ~ 0
+Text HLabel 9150 4200 0    50   BiDi ~ 0
 IO_L11_16_N
-Text HLabel 9950 4300 2    50   BiDi ~ 0
+Text HLabel 9950 4200 2    50   BiDi ~ 0
 IO_L11_16_P
 Wire Wire Line
-	9150 4300 9300 4300
+	9150 4200 9300 4200
+Wire Wire Line
+	9300 4300 9150 4300
+Wire Wire Line
+	9300 4500 9150 4500
+Wire Wire Line
+	9150 4600 9300 4600
+Wire Wire Line
+	9300 4800 9150 4800
+Wire Wire Line
+	9800 4800 9950 4800
+Wire Wire Line
+	9950 4600 9800 4600
+Wire Wire Line
+	9800 4500 9950 4500
+Wire Wire Line
+	9800 4300 9950 4300
+Wire Wire Line
+	9950 4200 9800 4200
+Text HLabel 9150 4600 0    50   BiDi ~ 0
+IO_L22_16_N
+Text HLabel 9950 4600 2    50   BiDi ~ 0
+IO_L22_16_P
+Wire Wire Line
+	9800 4400 9950 4400
 Wire Wire Line
 	9300 4400 9150 4400
-Wire Wire Line
-	9300 4600 9150 4600
-Wire Wire Line
-	9150 4700 9300 4700
-Wire Wire Line
-	9300 4800 9150 4800
-Wire Wire Line
-	9800 4800 9950 4800
-Wire Wire Line
-	9950 4700 9800 4700
-Wire Wire Line
-	9800 4600 9950 4600
-Wire Wire Line
-	9800 4400 9950 4400
-Wire Wire Line
-	9950 4300 9800 4300
-Text HLabel 9150 4700 0    50   BiDi ~ 0
-IO_L22_16_N
-Text HLabel 9950 4700 2    50   BiDi ~ 0
-IO_L22_16_P
-Wire Wire Line
-	9800 4500 9950 4500
-Wire Wire Line
-	9300 4500 9150 4500
 Wire Wire Line
 	9800 5700 9950 5700
@@
 Wire Wire Line
 	5300 3800 5150 3800
+Wire Wire Line
+	8550 4100 8550 4900
+Wire Wire Line
+	9300 4900 8550 4900
+Connection ~ 8550 4900
+Wire Wire Line
+	8550 4900 8550 5800
+Text HLabel 9950 4700 2    50   BiDi ~ 0
+IO_L23_16_P
+Text HLabel 9150 4700 0    50   BiDi ~ 0
+IO_L23_16_N
+Wire Wire Line
+	9300 4700 9150 4700
+Wire Wire Line
+	9800 4700 9950 4700
 $EndSCHEMATC

Commit message: v2 schematic/pcb progress commit - 12 unrouted
Connections:
- net IO_L23_16_N is gone; now on net IO_L22_16_N: J2.25 (Pin_25)
- net IO_L23_16_P is gone; now on net IO_L22_16_P: J2.26 (Pin_26)
- net IO_L11_16_N: now also J2.31 (Pin_31); no longer J2.35 (Pin_35)
- net IO_L11_16_P: now also J2.32 (Pin_32); no longer J2.36 (Pin_36)
- net IO_L20_16_N: now also J2.27 (Pin_27); no longer J2.29 (Pin_29)
- net IO_L20_16_P: now also J2.28 (Pin_28); no longer J2.30 (Pin_30)
- net IO_L21_16_N: now also J2.29 (Pin_29); no longer J2.31 (Pin_31)
- net IO_L21_16_P: now also J2.30 (Pin_30); no longer J2.32 (Pin_32)
- net IO_L22_16_N: no longer J2.27 (Pin_27)
- net IO_L22_16_P: no longer J2.28 (Pin_28)
- new net IO_L9_16_N: J2.35 (Pin_35)
- new net IO_L9_16_P: J2.36 (Pin_36)
Changed lines of the file:
@@
 Text HLabel 9150 4300 0    50   BiDi ~ 0
 IO_L17_16_N
-Text HLabel 9150 4400 0    50   BiDi ~ 0
+Text HLabel 9150 4500 0    50   BiDi ~ 0
 IO_L21_16_N
-Text HLabel 9950 4400 2    50   BiDi ~ 0
+Text HLabel 9950 4500 2    50   BiDi ~ 0
 IO_L21_16_P
-Text HLabel 9950 4500 2    50   BiDi ~ 0
+Text HLabel 9950 4600 2    50   BiDi ~ 0
 IO_L20_16_P
-Text HLabel 9150 4500 0    50   BiDi ~ 0
+Text HLabel 9150 4600 0    50   BiDi ~ 0
 IO_L20_16_N
 Text HLabel 9150 4800 0    50   BiDi ~ 0
@@
 Text HLabel 9950 4800 2    50   BiDi ~ 0
 IO_L24_16_P
-Text HLabel 9150 4200 0    50   BiDi ~ 0
+Text HLabel 9150 4400 0    50   BiDi ~ 0
 IO_L11_16_N
-Text HLabel 9950 4200 2    50   BiDi ~ 0
+Text HLabel 9950 4400 2    50   BiDi ~ 0
 IO_L11_16_P
 Wire Wire Line
-	9150 4200 9300 4200
-Wire Wire Line
-	9300 4300 9150 4300
+	9150 4300 9300 4300
+Wire Wire Line
+	9300 4400 9150 4400
+Wire Wire Line
+	9300 4600 9150 4600
+Wire Wire Line
+	9150 4700 9300 4700
+Wire Wire Line
+	9300 4800 9150 4800
+Wire Wire Line
+	9800 4800 9950 4800
+Wire Wire Line
+	9950 4700 9800 4700
+Wire Wire Line
+	9800 4600 9950 4600
+Wire Wire Line
+	9800 4400 9950 4400
+Wire Wire Line
+	9950 4300 9800 4300
+Text HLabel 9150 4700 0    50   BiDi ~ 0
+IO_L22_16_N
+Text HLabel 9950 4700 2    50   BiDi ~ 0
+IO_L22_16_P
+Wire Wire Line
+	9800 4500 9950 4500
 Wire Wire Line
 	9300 4500 9150 4500
-Wire Wire Line
-	9150 4600 9300 4600
-Wire Wire Line
-	9300 4800 9150 4800
-Wire Wire Line
-	9800 4800 9950 4800
-Wire Wire Line
-	9950 4600 9800 4600
-Wire Wire Line
-	9800 4500 9950 4500
-Wire Wire Line
-	9800 4300 9950 4300
-Wire Wire Line
-	9950 4200 9800 4200
-Text HLabel 9150 4600 0    50   BiDi ~ 0
-IO_L22_16_N
-Text HLabel 9950 4600 2    50   BiDi ~ 0
-IO_L22_16_P
-Wire Wire Line
-	9800 4400 9950 4400
-Wire Wire Line
-	9300 4400 9150 4400
 Wire Wire Line
 	9800 5700 9950 5700
@@
 Wire Wire Line
 	8550 4900 8550 5800
-Text HLabel 9950 4700 2    50   BiDi ~ 0
-IO_L23_16_P
-Text HLabel 9150 4700 0    50   BiDi ~ 0
-IO_L23_16_N
-Wire Wire Line
-	9300 4700 9150 4700
-Wire Wire Line
-	9800 4700 9950 4700
+Text HLabel 9150 4200 0    50   BiDi ~ 0
+IO_L9_16_N
+Text HLabel 9950 4200 2    50   BiDi ~ 0
+IO_L9_16_P
+Wire Wire Line
+	9950 4200 9800 4200
+Wire Wire Line
+	9300 4200 9150 4200
 $EndSCHEMATC

Commit message: v2 hardware: all tracks routed, erc/drc pass
Connections:
- net at U1.V20 (IO_L11N_T1_SRCC_14): now also TP8.1; no longer TP7.1
- net at U1.V22 (IO_L3N_T0_DQS_EMCCLK_14): now also TP7.1; no longer TP8.1
- no-connect marks 41 -> 42
Other:
- moved on the sheet: TP7, TP8
Changed lines of the file:
@@
 L tom-mechanical:TestPoint TP7
 U 1 1 5F3C3650
-P 5750 3900
-F 0 "TP7" V 5750 4088 50  0000 L CNN
-F 1 "TestPoint" H 5808 3927 50  0001 L CNN
-F 2 "tom-mechanical:TestPoint_Pad_D1.5mm" H 5950 3900 50  0001 C CNN
-F 3 "~" H 5950 3900 50  0001 C CNN
-	1    5750 3900
+P 5750 2300
+F 0 "TP7" V 5750 2488 50  0000 L CNN
+F 1 "TestPoint" H 5808 2327 50  0001 L CNN
+F 2 "tom-mechanical:TestPoint_Pad_D1.5mm" H 5950 2300 50  0001 C CNN
+F 3 "~" H 5950 2300 50  0001 C CNN
+	1    5750 2300
 	0    1    1    0
 $EndComp
@@
 Text HLabel 5300 3800 2    50   BiDi ~ 0
 IO_L11_14_P
-Wire Wire Line
-	5150 5700 5300 5700
 Text HLabel 4950 900  2    50   Input ~ 0
 VCCO_14
@@
 L tom-mechanical:TestPoint TP8
 U 1 1 5F3CB4AF
-P 5750 2300
-F 0 "TP8" V 5750 2488 50  0000 L CNN
-F 1 "TestPoint" H 5808 2327 50  0001 L CNN
-F 2 "tom-mechanical:TestPoint_Pad_D1.5mm" H 5950 2300 50  0001 C CNN
-F 3 "~" H 5950 2300 50  0001 C CNN
-	1    5750 2300
+P 5750 3900
+F 0 "TP8" V 5750 4088 50  0000 L CNN
+F 1 "TestPoint" H 5808 3927 50  0001 L CNN
+F 2 "tom-mechanical:TestPoint_Pad_D1.5mm" H 5950 3900 50  0001 C CNN
+F 3 "~" H 5950 3900 50  0001 C CNN
+	1    5750 3900
 	0    1    1    0
 $EndComp
@@
 Wire Wire Line
 	9300 4200 9150 4200
+NoConn ~ 5150 5700
 $EndSCHEMATC
