File: hardware/v2/artix7-pcie-v2-power.sch (KiCad schematic (older format))
At the start: 46 parts, among them U3 LP5907MFX, U5 TPS82130SILT, U6 TPS82150SILT, U7 TPS82150SILT, U8 TPS82130SILT, U9 TPS82150SILT

Commit message: v2 hardware: pcb progress commit, 155 unrouted
Parts:
- removed C17, C18: 22uF/25V/X5R, tom-passives:C_0603_1608Metric_Pad1.05x0.95mm_HandSolder, symbol tom-passives:C
- added R40, R41, R46, R47, R48, R49: 0R, tom-passives:C_0603_1608Metric, symbol tom-passives:R
- added R50: 0R, tom-passives:C_0402_1005Metric, symbol tom-passives:R
- C10, C35, C36, C39, C7: value 22uF/10V -> 22uF/6.3V/X7S; footprint tom-passives:C_0805_2012Metric -> tom-passives:C_1206_3216Metric
- C11, C13, C37, C5, C8: value 10uF/25V -> 10uF/25V/X7R
- R11, R15, R33: footprint tom-passives:R_0603_1608Metric -> tom-passives:C_0603_1608Metric
Connections:
- net +1V0: now also R46.1; no longer C7.1, R12.1, R14.2, U5.4 (VOUT), U5.5 (VOUT)
- net +1V8: now also R47.1; no longer C35.1, R22.1, R31.2, U7.4 (VOUT), U7.5 (VOUT)
- net +3V3: now also R48.1; no longer C39.1, R36.1, R39.2, U9.4 (VOUT), U9.5 (VOUT)
- net MGTAVTT: now also R50.1; no longer C14.1, U3.5 (OUT)
- net PG_1.8V: no longer U3.3 (EN)
- net VCCO_16: now also R49.1; no longer C10.1, R16.1, R18.2, U6.4 (VOUT), U6.5 (VOUT)
- net VCCO_34: now also R41.2; no longer C36.1, R24.1, R32.2, U8.4 (VOUT), U8.5 (VOUT)
- net PG_3.3V: now reaches R36.2, U9.7 (PG)
- net PG_3.3V: now also U3.3 (EN)
- net PG_16: now reaches R16.2, U6.7 (PG)
- new net VCCO_34_35: C36.1, R24.1, R32.2, R40.1, R41.1, U8.4 (VOUT), U8.5 (VOUT)
- new net VCCO_35: R40.2
- new net VOUT_1.8V: C35.1, R22.1, R31.2, R47.2, U7.4 (VOUT), U7.5 (VOUT)
- new net VOUT_16: C10.1, R16.1, R18.2, R49.2, U6.4 (VOUT), U6.5 (VOUT)
- new net VOUT_1V: C7.1, R12.1, R14.2, R46.2, U5.4 (VOUT), U5.5 (VOUT)
- new net VOUT_3.3V: C39.1, R36.1, R39.2, R48.2, U9.4 (VOUT), U9.5 (VOUT)
- new net VOUT_MGTAVTT: C14.1, R50.2, U3.5 (OUT)
Other:
- note added: "Sequence #4 1.2V\nVTT (156mA est)"
- note removed: "Sequence #3 1.2V\nVTT (156mA est)"

Commit message: v2 hardware: j2_34 diff pairs matched, fix 0402 resistor packages, dropped paste from DNP resistors
Parts:
- R11, R15, R33, R40, R41, R46, R47, R48, R49: footprint tom-passives:C_0603_1608Metric -> tom-passives:R_0603_1608Metric_NoPaste
- R12, R13, R14, R16, R17, R18, R22, R23, R24, R25, R31, R32, R36, R38, R39: footprint tom-passives:C_0402_1005Metric -> tom-passives:R_0402_1005Metric
- R19, R21: footprint tom-passives:R_0603_1608Metric -> tom-passives:R_0603_1608Metric_NoPaste
- R20, R50: footprint tom-passives:C_0402_1005Metric -> tom-passives:R_0402_1005Metric_NoPaste
Changed lines of the file:
@@
 F 0 "R20" H 8471 3938 40  0000 L CNN
 F 1 "0R" H 8471 3862 40  0000 L CNN
-F 2 "tom-passives:C_0402_1005Metric" H 8471 3824 30  0001 L CNN
+F 2 "tom-passives:R_0402_1005Metric_NoPaste" H 8471 3824 30  0001 L CNN
 F 3 "" H 8400 3900 30  0001 C CNN
 	1    8400 3900
@@
 F 0 "R13" H 3071 2138 40  0000 L CNN
 F 1 "100k/1%" H 3071 2062 40  0000 L CNN
-F 2 "tom-passives:C_0402_1005Metric" V 2930 2100 30  0001 C CNN
+F 2 "tom-passives:R_0402_1005Metric" V 2930 2100 30  0001 C CNN
 F 3 "" H 3000 2100 30  0001 C CNN
 	1    3000 2100
@@
 F 0 "R14" V 3435 1750 40  0000 C CNN
 F 1 "24.9k/1%" V 3359 1750 40  0000 C CNN
-F 2 "tom-passives:C_0402_1005Metric" V 3180 1750 30  0001 C CNN
+F 2 "tom-passives:R_0402_1005Metric" V 3180 1750 30  0001 C CNN
 F 3 "" H 3250 1750 30  0001 C CNN
 	1    3250 1750
@@
 F 0 "R12" H 3071 1088 40  0000 L CNN
 F 1 "100k/5%" H 3071 1012 40  0000 L CNN
-F 2 "tom-passives:C_0402_1005Metric" H 3071 974 30  0001 L CNN
+F 2 "tom-passives:R_0402_1005Metric" H 3071 974 30  0001 L CNN
 F 3 "" H 3000 1050 30  0001 C CNN
 	1    3000 1050
@@
 F 0 "R23" H 6521 2138 40  0000 L CNN
 F 1 "100k/1%" H 6521 2062 40  0000 L CNN
-F 2 "tom-passives:C_0402_1005Metric" V 6380 2100 30  0001 C CNN
+F 2 "tom-passives:R_0402_1005Metric" V 6380 2100 30  0001 C CNN
 F 3 "" H 6450 2100 30  0001 C CNN
 	1    6450 2100
@@
 F 0 "R31" V 6885 1750 40  0000 C CNN
 F 1 "124k/1%" V 6809 1750 40  0000 C CNN
-F 2 "tom-passives:C_0402_1005Metric" V 6630 1750 30  0001 C CNN
+F 2 "tom-passives:R_0402_1005Metric" V 6630 1750 30  0001 C CNN
 F 3 "" H 6700 1750 30  0001 C CNN
 	1    6700 1750
@@
 F 0 "R22" H 6521 1088 40  0000 L CNN
 F 1 "100k/5%" H 6521 1012 40  0000 L CNN
-F 2 "tom-passives:C_0402_1005Metric" H 6521 974 30  0001 L CNN
+F 2 "tom-passives:R_0402_1005Metric" H 6521 974 30  0001 L CNN
 F 3 "" H 6450 1050 30  0001 C CNN
 	1    6450 1050
@@
 F 0 "R33" H 8071 1038 40  0000 L CNN
 F 1 "0R" H 8071 962 40  0000 L CNN
-F 2 "tom-passives:C_0603_1608Metric" H 8071 924 30  0001 L CNN
+F 2 "tom-passives:R_0603_1608Metric_NoPaste" H 8071 924 30  0001 L CNN
 F 3 "" H 8000 1000 30  0001 C CNN
 	1    8000 1000
@@
 F 0 "R38" H 10121 2138 40  0000 L CNN
 F 1 "100k/1%" H 10121 2062 40  0000 L CNN
-F 2 "tom-passives:C_0402_1005Metric" V 9980 2100 30  0001 C CNN
+F 2 "tom-passives:R_0402_1005Metric" V 9980 2100 30  0001 C CNN
 F 3 "" H 10050 2100 30  0001 C CNN
 	1    10050 2100
@@
 F 0 "R39" V 10485 1750 40  0000 C CNN
 F 1 "316k/1%" V 10409 1750 40  0000 C CNN
-F 2 "tom-passives:C_0402_1005Metric" V 10230 1750 30  0001 C CNN
+F 2 "tom-passives:R_0402_1005Metric" V 10230 1750 30  0001 C CNN
 F 3 "" H 10300 1750 30  0001 C CNN
 	1    10300 1750
@@
 F 0 "R15" H 1021 3788 40  0000 L CNN
 F 1 "0R" H 1021 3712 40  0000 L CNN
-F 2 "tom-passives:C_0603_1608Metric" H 1021 3674 30  0001 L CNN
+F 2 "tom-passives:R_0603_1608Metric_NoPaste" H 1021 3674 30  0001 L CNN
 F 3 "" H 950 3750 30  0001 C CNN
 	1    950  3750
@@
 F 0 "R17" H 3071 4888 40  0000 L CNN
 F 1 "100k/1%" H 3071 4812 40  0000 L CNN
-F 2 "tom-passives:C_0402_1005Metric" V 2930 4850 30  0001 C CNN
+F 2 "tom-passives:R_0402_1005Metric" V 2930 4850 30  0001 C CNN
 F 3 "" H 3000 4850 30  0001 C CNN
 	1    3000 4850
@@
 F 0 "R18" V 3435 4500 40  0000 C CNN
 F 1 "213k/1%" V 3359 4500 40  0000 C CNN
-F 2 "tom-passives:C_0402_1005Metric" V 3180 4500 30  0001 C CNN
+F 2 "tom-passives:R_0402_1005Metric" V 3180 4500 30  0001 C CNN
 F 3 "" H 3250 4500 30  0001 C CNN
 	1    3250 4500
@@
 F 0 "R16" H 3071 3838 40  0000 L CNN
 F 1 "100k/5%" H 3071 3762 40  0000 L CNN
-F 2 "tom-passives:C_0402_1005Metric" H 3071 3724 30  0001 L CNN
+F 2 "tom-passives:R_0402_1005Metric" H 3071 3724 30  0001 L CNN
 F 3 "" H 3000 3800 30  0001 C CNN
 	1    3000 3800
@@
 F 0 "R21" H 4471 3788 40  0000 L CNN
 F 1 "0R" H 4471 3712 40  0000 L CNN
-F 2 "tom-passives:R_0603_1608Metric" H 4471 3674 30  0001 L CNN
+F 2 "tom-passives:R_0603_1608Metric_NoPaste" H 4471 3674 30  0001 L CNN
 F 3 "" H 4400 3750 30  0001 C CNN
 	1    4400 3750
@@
 F 0 "R25" H 6521 4888 40  0000 L CNN
 F 1 "100k/1%" H 6521 4812 40  0000 L CNN
-F 2 "tom-passives:C_0402_1005Metric" V 6380 4850 30  0001 C CNN
+F 2 "tom-passives:R_0402_1005Metric" V 6380 4850 30  0001 C CNN
 F 3 "" H 6450 4850 30  0001 C CNN
 	1    6450 4850
@@
 F 0 "R32" V 6885 4500 40  0000 C CNN
 F 1 "124k/1%" V 6809 4500 40  0000 C CNN
-F 2 "tom-passives:C_0402_1005Metric" V 6630 4500 30  0001 C CNN
+F 2 "tom-passives:R_0402_1005Metric" V 6630 4500 30  0001 C CNN
 F 3 "" H 6700 4500 30  0001 C CNN
 	1    6700 4500
@@
 F 0 "R24" H 6521 3838 40  0000 L CNN
 F 1 "100k/5%" H 6521 3762 40  0000 L CNN
-F 2 "tom-passives:C_0402_1005Metric" H 6521 3724 30  0001 L CNN
+F 2 "tom-passives:R_0402_1005Metric" H 6521 3724 30  0001 L CNN
 F 3 "" H 6450 3800 30  0001 C CNN
 	1    6450 3800
@@
 F 0 "R40" H 1921 6988 40  0000 L CNN
 F 1 "0R" H 1921 6912 40  0000 L CNN
-F 2 "tom-passives:C_0603_1608Metric" H 1921 6874 30  0001 L CNN
+F 2 "tom-passives:R_0603_1608Metric_NoPaste" H 1921 6874 30  0001 L CNN
 F 3 "" H 1850 6950 30  0001 C CNN
 	1    1850 6950
@@
 F 0 "R41" H 2271 6788 40  0000 L CNN
 F 1 "0R" H 2271 6712 40  0000 L CNN
-F 2 "tom-passives:C_0603_1608Metric" H 2271 6674 30  0001 L CNN
+F 2 "tom-passives:R_0603_1608Metric_NoPaste" H 2271 6674 30  0001 L CNN
 F 3 "" H 2200 6750 30  0001 C CNN
 	1    2200 6750
@@
 F 0 "R46" H 3821 838 40  0000 L CNN
 F 1 "0R" H 3821 762 40  0000 L CNN
-F 2 "tom-passives:C_0603_1608Metric" H 3821 724 30  0001 L CNN
+F 2 "tom-passives:R_0603_1608Metric_NoPaste" H 3821 724 30  0001 L CNN
 F 3 "" H 3750 800 30  0001 C CNN
 	1    3750 800
@@
 F 0 "R47" H 7271 838 40  0000 L CNN
 F 1 "0R" H 7271 762 40  0000 L CNN
-F 2 "tom-passives:C_0603_1608Metric" H 7271 724 30  0001 L CNN
+F 2 "tom-passives:R_0603_1608Metric_NoPaste" H 7271 724 30  0001 L CNN
 F 3 "" H 7200 800 30  0001 C CNN
 	1    7200 800
@@
 F 0 "R48" H 10871 1488 40  0000 L CNN
 F 1 "0R" H 10871 1412 40  0000 L CNN
-F 2 "tom-passives:C_0603_1608Metric" H 10871 1374 30  0001 L CNN
+F 2 "tom-passives:R_0603_1608Metric_NoPaste" H 10871 1374 30  0001 L CNN
 F 3 "" H 10800 1450 30  0001 C CNN
 	1    10800 1450
@@
 F 0 "R49" H 3771 3988 40  0000 L CNN
 F 1 "0R" H 3771 3912 40  0000 L CNN
-F 2 "tom-passives:C_0603_1608Metric" H 3771 3874 30  0001 L CNN
+F 2 "tom-passives:R_0603_1608Metric_NoPaste" H 3771 3874 30  0001 L CNN
 F 3 "" H 3700 3950 30  0001 C CNN
 	1    3700 3950
@@
 F 0 "R50" H 10121 4188 40  0000 L CNN
 F 1 "0R" H 10121 4112 40  0000 L CNN
-F 2 "tom-passives:C_0402_1005Metric" H 10121 4074 30  0001 L CNN
+F 2 "tom-passives:R_0402_1005Metric_NoPaste" H 10121 4074 30  0001 L CNN
 F 3 "" H 10050 4150 30  0001 C CNN
 	1    10050 4150
@@
 F 0 "R19" H 4471 1038 40  0000 L CNN
 F 1 "0R" H 4471 962 40  0000 L CNN
-F 2 "tom-passives:R_0603_1608Metric" H 4471 924 30  0001 L CNN
+F 2 "tom-passives:R_0603_1608Metric_NoPaste" H 4471 924 30  0001 L CNN
 F 3 "" H 4400 1000 30  0001 C CNN
 	1    4400 1000
@@
 F 0 "R11" H 1021 1038 40  0000 L CNN
 F 1 "0R" H 1021 962 40  0000 L CNN
-F 2 "tom-passives:C_0603_1608Metric" H 1021 924 30  0001 L CNN
+F 2 "tom-passives:R_0603_1608Metric_NoPaste" H 1021 924 30  0001 L CNN
 F 3 "" H 950 1000 30  0001 C CNN
 	1    950  1000
@@
 F 0 "R36" H 10121 1088 40  0000 L CNN
 F 1 "100k/5%" H 10121 1012 40  0000 L CNN
-F 2 "tom-passives:C_0402_1005Metric" H 10121 974 30  0001 L CNN
+F 2 "tom-passives:R_0402_1005Metric" H 10121 974 30  0001 L CNN
 F 3 "" H 10050 1050 30  0001 C CNN
 	1    10050 1050

Commit message: v2 hardware: add Digikey part numbers to schematic and generate bom
Parts:
- C10, C35, C36, C39, C7: Vendor (none) -> 1276-1771-1-ND
- C11, C13, C37, C5, C8: Vendor (none) -> 399-8153-1-ND
- C15, C16, C38, C6, C9: Vendor (none) -> 490-3248-1-ND
- R12, R16, R22, R24, R36: value 100k/5% -> 100k/1%
- R14: Vendor (none) -> RMCF0402FT24K9CT-ND
- R18: value 213k/1% -> 215k/1%; Vendor (none) -> RMCF0402FT215KCT-ND
- R31, R32: Vendor (none) -> 2019-RK73H1ETTP1243FCT-ND
- R39: Vendor (none) -> 738-RMCF0402FT316KCT-ND
- U3: Vendor (none) -> 296-LP5907UVX-1.2/NOPBCT-ND
- U5, U8: Vendor (none) -> 296-47436-1-ND
- U6, U7, U9: Vendor (none) -> 296-47090-1-ND
Other:
- note added: "0.8 * (1+215/100) =2.52V"
- note removed: "0.8 * (1+213/100) =2.504V"
Changed lines of the file:
@@
 F 2 "tom-semiconductors:SOT-23-5" H 9300 4250 50  0001 C CNN
 F 3 "http://www.ti.com/lit/ds/symlink/lp5907.pdf" H 9300 4250 50  0001 C CNN
+F 4 "296-LP5907UVX-1.2/NOPBCT-ND" H 9300 4250 50  0001 C CNN "Vendor"
 	1    9300 4250
 	1    0    0    -1
@@
 F 3 "" H 950 1550 60  0001 C CNN
 F 4 "C3216X7R1E106M160AE" H 950 1550 50  0001 C CNN "MFGPN"
+F 5 "399-8153-1-ND" H 950 1550 50  0001 C CNN "Vendor"
 	1    950  1550
 	1    0    0    1
@@
 F 2 "tom-passives:C_0402_1005Metric" H 1286 2126 30  0001 R CNN
 F 3 "" H 1400 2050 60  0001 C CNN
+F 4 "490-3248-1-ND" H 1400 2050 50  0001 C CNN "Vendor"
 	1    1400 2050
 	1    0    0    1
@@
 F 2 "tom-passives:R_0402_1005Metric" V 3180 1750 30  0001 C CNN
 F 3 "" H 3250 1750 30  0001 C CNN
+F 4 "RMCF0402FT24K9CT-ND" H 3250 1750 50  0001 C CNN "Vendor"
 	1    3250 1750
 	0    -1   -1   0
@@
 P 3000 1050
 F 0 "R12" H 3071 1088 40  0000 L CNN
-F 1 "100k/5%" H 3071 1012 40  0000 L CNN
+F 1 "100k/1%" H 3071 1012 40  0000 L CNN
 F 2 "tom-passives:R_0402_1005Metric" H 3071 974 30  0001 L CNN
 F 3 "" H 3000 1050 30  0001 C CNN
@@
 F 3 "" H 3500 1950 60  0001 C CNN
 F 4 "C2012X7S1A226M125AC" H 3500 1950 50  0001 C CNN "MFGPN"
+F 5 "1276-1771-1-ND" H 3500 1950 50  0001 C CNN "Vendor"
 	1    3500 1950
 	1    0    0    -1
@@
 F 3 "" H 4400 1550 60  0001 C CNN
 F 4 "C3216X7R1E106M160AE" H 4400 1550 50  0001 C CNN "MFGPN"
+F 5 "399-8153-1-ND" H 4400 1550 50  0001 C CNN "Vendor"
 	1    4400 1550
 	1    0    0    1
@@
 F 2 "tom-passives:C_0402_1005Metric" H 4736 2126 30  0001 R CNN
 F 3 "" H 4850 2050 60  0001 C CNN
+F 4 "490-3248-1-ND" H 4850 2050 50  0001 C CNN "Vendor"
 	1    4850 2050
 	1    0    0    1
@@
 F 2 "tom-passives:R_0402_1005Metric" V 6630 1750 30  0001 C CNN
 F 3 "" H 6700 1750 30  0001 C CNN
+F 4 "2019-RK73H1ETTP1243FCT-ND" H 6700 1750 50  0001 C CNN "Vendor"
 	1    6700 1750
 	0    -1   -1   0
@@
 P 6450 1050
 F 0 "R22" H 6521 1088 40  0000 L CNN
-F 1 "100k/5%" H 6521 1012 40  0000 L CNN
+F 1 "100k/1%" H 6521 1012 40  0000 L CNN
 F 2 "tom-passives:R_0402_1005Metric" H 6521 974 30  0001 L CNN
 F 3 "" H 6450 1050 30  0001 C CNN
@@
 F 3 "" H 6950 1950 60  0001 C CNN
 F 4 "C2012X7S1A226M125AC" H 6950 1950 50  0001 C CNN "MFGPN"
+F 5 "1276-1771-1-ND" H 6950 1950 50  0001 C CNN "Vendor"
 	1    6950 1950
 	1    0    0    -1
@@
 F 2 "tom-modules:TPS82130SILT" H 9250 1640 60  0001 C CNN
 F 3 "http://www.ti.com/lit/ds/symlink/tps82130.pdf" H 9250 1701 60  0001 C CNN
+F 4 "296-47090-1-ND" H 8450 1400 50  0001 C CNN "Vendor"
 	1    8450 1400
 	1    0    0    -1
@@
 F 3 "" H 8000 1550 60  0001 C CNN
 F 4 "C3216X7R1E106M160AE" H 8000 1550 50  0001 C CNN "MFGPN"
+F 5 "399-8153-1-ND" H 8000 1550 50  0001 C CNN "Vendor"
 	1    8000 1550
 	1    0    0    1
@@
 F 2 "tom-passives:C_0402_1005Metric" H 8336 2126 30  0001 R CNN
 F 3 "" H 8450 2050 60  0001 C CNN
+F 4 "490-3248-1-ND" H 8450 2050 50  0001 C CNN "Vendor"
 	1    8450 2050
 	1    0    0    1
@@
 F 2 "tom-passives:R_0402_1005Metric" V 10230 1750 30  0001 C CNN
 F 3 "" H 10300 1750 30  0001 C CNN
+F 4 "738-RMCF0402FT316KCT-ND" H 10300 1750 50  0001 C CNN "Vendor"
 	1    10300 1750
 	0    -1   -1   0
@@
 F 3 "" H 10550 1950 60  0001 C CNN
 F 4 "C2012X7S1A226M125AC" H 10550 1950 50  0001 C CNN "MFGPN"
+F 5 "1276-1771-1-ND" H 10550 1950 50  0001 C CNN "Vendor"
 	1    10550 1950
 	1    0    0    -1
@@
 F 2 "tom-modules:TPS82130SILT" H 2200 4390 60  0001 C CNN
 F 3 "http://www.ti.com/lit/ds/symlink/tps82130.pdf" H 2200 4451 60  0001 C CNN
+F 4 "296-47090-1-ND" H 1400 4150 50  0001 C CNN "Vendor"
 	1    1400 4150
 	1    0    0    -1
@@
 F 3 "" H 950 4300 60  0001 C CNN
 F 4 "C3216X7R1E106M160AE" H 950 4300 50  0001 C CNN "MFGPN"
+F 5 "399-8153-1-ND" H 950 4300 50  0001 C CNN "Vendor"
 	1    950  4300
 	1    0    0    1
@@
 F 2 "tom-passives:C_0402_1005Metric" H 1286 4876 30  0001 R CNN
 F 3 "" H 1400 4800 60  0001 C CNN
+F 4 "490-3248-1-ND" H 1400 4800 50  0001 C CNN "Vendor"
 	1    1400 4800
 	1    0    0    1
@@
 P 3250 4500
 F 0 "R18" V 3435 4500 40  0000 C CNN
-F 1 "213k/1%" V 3359 4500 40  0000 C CNN
+F 1 "215k/1%" V 3359 4500 40  0000 C CNN
 F 2 "tom-passives:R_0402_1005Metric" V 3180 4500 30  0001 C CNN
 F 3 "" H 3250 4500 30  0001 C CNN
+F 4 "RMCF0402FT215KCT-ND" H 3250 4500 50  0001 C CNN "Vendor"
 	1    3250 4500
 	0    -1   -1   0
@@
 P 3000 3800
 F 0 "R16" H 3071 3838 40  0000 L CNN
-F 1 "100k/5%" H 3071 3762 40  0000 L CNN
+F 1 "100k/1%" H 3071 3762 40  0000 L CNN
 F 2 "tom-passives:R_0402_1005Metric" H 3071 3724 30  0001 L CNN
 F 3 "" H 3000 3800 30  0001 C CNN
@@
 F 3 "" H 3500 4700 60  0001 C CNN
 F 4 "C2012X7S1A226M125AC" H 3500 4700 50  0001 C CNN "MFGPN"
+F 5 "1276-1771-1-ND" H 3500 4700 50  0001 C CNN "Vendor"
 	1    3500 4700
 	1    0    0    -1
@@
 $EndComp
 Text Notes 1600 5350 0    50   ~ 0
-0.8 * (1+213/100) =2.504V
+0.8 * (1+215/100) =2.52V
 Wire Wire Line
 	950  4100 1400 4100
@@
 F 2 "tom-modules:TPS82130SILT" H 5650 4390 60  0001 C CNN
 F 3 "http://www.ti.com/lit/ds/symlink/tps82130.pdf" H 5650 4451 60  0001 C CNN
+F 4 "296-47436-1-ND" H 4850 4150 50  0001 C CNN "Vendor"
 	1    4850 4150
 	1    0    0    -1
@@
 F 3 "" H 4400 4300 60  0001 C CNN
 F 4 "C3216X7R1E106M160AE" H 4400 4300 50  0001 C CNN "MFGPN"
+F 5 "399-8153-1-ND" H 4400 4300 50  0001 C CNN "Vendor"
 	1    4400 4300
 	1    0    0    1
@@
 F 2 "tom-passives:C_0402_1005Metric" H 4736 4876 30  0001 R CNN
 F 3 "" H 4850 4800 60  0001 C CNN
+F 4 "490-3248-1-ND" H 4850 4800 50  0001 C CNN "Vendor"
 	1    4850 4800
 	1    0    0    1
@@
 F 2 "tom-passives:R_0402_1005Metric" V 6630 4500 30  0001 C CNN
 F 3 "" H 6700 4500 30  0001 C CNN
+F 4 "2019-RK73H1ETTP1243FCT-ND" H 6700 4500 50  0001 C CNN "Vendor"
 	1    6700 4500
 	0    -1   -1   0
@@
 P 6450 3800
 F 0 "R24" H 6521 3838 40  0000 L CNN
-F 1 "100k/5%" H 6521 3762 40  0000 L CNN
+F 1 "100k/1%" H 6521 3762 40  0000 L CNN
 F 2 "tom-passives:R_0402_1005Metric" H 6521 3724 30  0001 L CNN
 F 3 "" H 6450 3800 30  0001 C CNN
@@
 F 3 "" H 6950 4700 60  0001 C CNN
 F 4 "C2012X7S1A226M125AC" H 6950 4700 50  0001 C CNN "MFGPN"
+F 5 "1276-1771-1-ND" H 6950 4700 50  0001 C CNN "Vendor"
 	1    6950 4700
 	1    0    0    -1
@@
 F 2 "tom-modules:TPS82130SILT" H 5650 1640 60  0001 C CNN
 F 3 "http://www.ti.com/lit/ds/symlink/tps82130.pdf" H 5650 1701 60  0001 C CNN
+F 4 "296-47090-1-ND" H 4850 1400 50  0001 C CNN "Vendor"
 	1    4850 1400
 	1    0    0    -1
@@
 F 2 "tom-modules:TPS82130SILT" H 2200 1640 60  0001 C CNN
 F 3 "http://www.ti.com/lit/ds/symlink/tps82130.pdf" H 2200 1701 60  0001 C CNN
+F 4 "296-47436-1-ND" H 1400 1400 50  0001 C CNN "Vendor"
 	1    1400 1400
 	1    0    0    -1
@@
 P 10050 1050
 F 0 "R36" H 10121 1088 40  0000 L CNN
-F 1 "100k/5%" H 10121 1012 40  0000 L CNN
+F 1 "100k/1%" H 10121 1012 40  0000 L CNN
 F 2 "tom-passives:R_0402_1005Metric" H 10121 974 30  0001 L CNN
 F 3 "" H 10050 1050 30  0001 C CNN

Commit message: hardware v2: bom fixes
Parts:
- U3: Vendor 296-LP5907UVX-1.2/NOPBCT-ND -> ‎296-39062-1-ND‎
Changed lines of the file:
@@
 F 2 "tom-semiconductors:SOT-23-5" H 9300 4250 50  0001 C CNN
 F 3 "http://www.ti.com/lit/ds/symlink/lp5907.pdf" H 9300 4250 50  0001 C CNN
-F 4 "296-LP5907UVX-1.2/NOPBCT-ND" H 9300 4250 50  0001 C CNN "Vendor"
+F 4 "‎296-39062-1-ND‎" H 9300 4250 50  0001 C CNN "Vendor"
 	1    9300 4250
 	1    0    0    -1

Commit message: hardware v2: fix digikey part number for U3
Parts:
- U3: Vendor ‎296-39062-1-ND‎ -> 296-40359-1-ND
Changed lines of the file:
@@
 F 2 "tom-semiconductors:SOT-23-5" H 9300 4250 50  0001 C CNN
 F 3 "http://www.ti.com/lit/ds/symlink/lp5907.pdf" H 9300 4250 50  0001 C CNN
-F 4 "‎296-39062-1-ND‎" H 9300 4250 50  0001 C CNN "Vendor"
+F 4 "296-40359-1-ND" H 9300 4250 50  0001 C CNN "Vendor"
 	1    9300 4250
 	1    0    0    -1

Commit message: hardware v2: fix digikey part number on MGTAVTT regulator
Parts:
- U3: Vendor 296-40359-1-ND -> 296-39062-1-ND
Changed lines of the file:
@@
 F 2 "tom-semiconductors:SOT-23-5" H 9300 4250 50  0001 C CNN
 F 3 "http://www.ti.com/lit/ds/symlink/lp5907.pdf" H 9300 4250 50  0001 C CNN
-F 4 "296-40359-1-ND" H 9300 4250 50  0001 C CNN "Vendor"
+F 4 "296-39062-1-ND" H 9300 4250 50  0001 C CNN "Vendor"
 	1    9300 4250
 	1    0    0    -1

Commit message: v2 hardware: aug2020 pcb updates
Parts:
- removed R11, R15, R19, R21, R33, R46, R47, R48, R49: 0R, tom-passives:R_0603_1608Metric_NoPaste, symbol tom-passives:R
- removed R20, R50: 0R, tom-passives:R_0402_1005Metric_NoPaste, symbol tom-passives:R
Connections:
- net VIN_1.0V is gone; now on net VCC: C5.2, U5.1 (EN), U5.2 (VIN)
- net VIN_1.8V is gone; now on net VCC: C11.2, U7.2 (VIN)
- net VIN_16 is gone; now on net VCC: C8.2, U6.2 (VIN)
- net VIN_3.3V is gone; now on net VCC: C37.2, U9.2 (VIN)
- net VIN_34_35 is gone; now on net VCC: C13.2, U8.2 (VIN)
- net VIN_MGTAVTT is gone; now on net +3V3: C12.1, U3.1 (IN)
- net VOUT_1.8V is gone; now on net +1V8: C35.1, R22.1, R31.2, U7.4 (VOUT), U7.5 (VOUT)
- net VOUT_16 is gone; now on net VCCO_16: C10.1, R16.1, R18.2, U6.4 (VOUT), U6.5 (VOUT)
- net VOUT_1V is gone; now on net +1V0: C7.1, R12.1, R14.2, U5.4 (VOUT), U5.5 (VOUT)
- net VOUT_3.3V is gone; now on net +3V3: C39.1, R36.1, R39.2, U9.4 (VOUT), U9.5 (VOUT)
- net VOUT_MGTAVTT is gone; now on net MGTAVTT: C14.1, U3.5 (OUT)
