File: hardware/v2/artix7-pcie-v2-bank15.sch (KiCad schematic (older format))
At the start: 10 parts, among them U1 XC7A75T-FGG484

Commit message: v2 hardware: Aug2020/rc2 version - flip tx/rx pairs on s2 - add lcsc part numbers
rc2 errata schematic
- change serial port connector to add +3.3V ? (8-pin)(NO)
- add test points for flash pre-programming
- smaller package on input direction diodes (NO)
- bom dupe errors
- remove all p/s 0R bringup parts
- optimise bom (use 1.5k for led, 10k/4.7k for i2c pullups)
- done led is bright (change to 4.7k)
- improve shield grounding with RC
- check actual values of RGB resistors
- remove caps from clock inputs

rc2 errata pcb
- no gnd marking on serial port connector pins
- change serial port connector to add +3.3V ? (8-pin) (NO)
- no test points for flash pre-programming
- missing caps on xtal? (No but select xtal carefully)
- Cfg sel pins on clock chip?
- No silk on test points
- No +/- pair numbering on silk
- vcc test points for clk pre-programming? (or use bootloader)
- random silk circle under S2
- smaller package on input direction diodes (NO)
- no polarity on 100uF tantalum
- some via in or close to pads
- wrong button package (change from feather to chinese)
- gnd/vcc labels swapped at high end of J2
- clock chip OUT0_SEL_I2CB needs to be tied high after programming
- check teardrops
- power diode footprint marking reverse
- LEDs use cap footprint
Parts:
- C78: LCSC (none) -> C15008
- C79, C80: LCSC (none) -> C23733
- C81, C82, C83, C84: LCSC (none) -> C47339
- TP5, TP6, U1: LCSC (none) -> DNP
Changed lines of the file:
@@
 F 2 "artix7-pcie-v2:Xilinx_FGG484" H 2550 4400 50  0001 C CNN
 F 3 "" H 2550 4400 50  0000 C CNN
+F 4 "DNP" H 2550 4400 50  0001 C CNN "LCSC"
 	2    2550 4400
 	1    0    0    -1
@@
 F 2 "tom-mechanical:TestPoint_Pad_D1.5mm" H 4758 3527 50  0001 L CNN
 F 3 "~" H 4900 3500 50  0001 C CNN
+F 4 "DNP" H 4700 3500 50  0001 C CNN "LCSC"
 	1    4700 3500
 	1    0    0    -1
@@
 F 2 "tom-mechanical:TestPoint_Pad_D1.5mm" H 5008 3527 50  0001 L CNN
 F 3 "~" H 5150 3500 50  0001 C CNN
+F 4 "DNP" H 4950 3500 50  0001 C CNN "LCSC"
 	1    4950 3500
 	1    0    0    -1
@@
 F 3 "" H 8450 2000 60  0001 C CNN
 F 4 "478-12404-1-ND" H 8450 2000 50  0001 C CNN "Vendor"
+F 5 "C15008" H 8450 2000 50  0001 C CNN "LCSC"
 	1    8450 2000
 	1    0    0    -1
@@
 F 3 "" H 8650 2000 60  0001 C CNN
 F 4 "490-5915-1-ND" H 8650 2000 50  0001 C CNN "Vendor"
+F 5 "C23733" H 8650 2000 50  0001 C CNN "LCSC"
 	1    8650 2000
 	1    0    0    -1
@@
 F 3 "" H 8850 2000 60  0001 C CNN
 F 4 "490-5915-1-ND" H 8850 2000 50  0001 C CNN "Vendor"
+F 5 "C23733" H 8850 2000 50  0001 C CNN "LCSC"
 	1    8850 2000
 	1    0    0    -1
@@
 F 3 "" H 9050 2000 60  0001 C CNN
 F 4 "1276-CL05Y474KP5VPNCCT-ND" H 9050 2000 50  0001 C CNN "Vendor"
+F 5 "C47339" H 9050 2000 50  0001 C CNN "LCSC"
 	1    9050 2000
 	1    0    0    -1
@@
 F 3 "" H 9250 2000 60  0001 C CNN
 F 4 "1276-CL05Y474KP5VPNCCT-ND" H 9250 2000 50  0001 C CNN "Vendor"
+F 5 "C47339" H 9250 2000 50  0001 C CNN "LCSC"
 	1    9250 2000
 	1    0    0    -1
@@
 F 3 "" H 9450 2000 60  0001 C CNN
 F 4 "1276-CL05Y474KP5VPNCCT-ND" H 9450 2000 50  0001 C CNN "Vendor"
+F 5 "C47339" H 9450 2000 50  0001 C CNN "LCSC"
 	1    9450 2000
 	1    0    0    -1
@@
 F 3 "" H 9650 2000 60  0001 C CNN
 F 4 "1276-CL05Y474KP5VPNCCT-ND" H 9650 2000 50  0001 C CNN "Vendor"
+F 5 "C47339" H 9650 2000 50  0001 C CNN "LCSC"
 	1    9650 2000
 	1    0    0    -1

Commit message: v2 hardware: change 100uF to 3528 for jlcpcb
Parts:
- C78: footprint tom-passives:CP_EIA-3216-12_Kemet-S -> tom-passives:CP_EIA-3528-15_AVX-H
Changed lines of the file:
@@
 F 0 "C78" V 8400 1200 40  0000 L CNN
 F 1 "100uF/6.3V/X5R" V 8500 1200 40  0000 L CNN
-F 2 "tom-passives:CP_EIA-3216-12_Kemet-S" H 8488 1850 30  0001 C CNN
+F 2 "tom-passives:CP_EIA-3528-15_AVX-H" H 8488 1850 30  0001 C CNN
 F 3 "" H 8450 2000 60  0001 C CNN
 F 4 "478-12404-1-ND" H 8450 2000 50  0001 C CNN "Vendor"

Commit message: v2 hardware: sep2020 run - fixed issues with parts missing from centroid file
Parts:
- C78: LCSC C15008 -> C16133
Changed lines of the file:
@@
 F 3 "" H 8450 2000 60  0001 C CNN
 F 4 "478-12404-1-ND" H 8450 2000 50  0001 C CNN "Vendor"
-F 5 "C15008" H 8450 2000 50  0001 C CNN "LCSC"
+F 5 "C16133" H 8450 2000 50  0001 C CNN "LCSC"
 	1    8450 2000
 	1    0    0    -1
