File: hardware/v2/artix7-pcie-v2-bank34.sch (KiCad schematic (older format))
At the start: 22 parts, among them J1 Conn_02x20_Odd_Even, U1 XC7A75T-FGG484

Commit message: v2 hardware: aug2020 pcb updates
Parts:
- C18, C23, C85, C86: footprint tom-passives:C_1206_3216Metric -> tom-passives:CP_EIA-3216-12_Kemet-S; symbol tom-passives:C -> tom-passives:CP_Small
Changed lines of the file:
@@
 VCCO_34
 $Comp
-L tom-passives:C C?
+L tom-passives:CP_Small C?
 U 1 1 5E9ED7A0
 P 6900 1200
@@
 F 0 "C85" V 6850 400 40  0000 L CNN
 F 1 "100uF/6.3V/X5R" V 6950 400 40  0000 L CNN
-F 2 "tom-passives:C_1206_3216Metric" H 6938 1050 30  0001 C CNN
+F 2 "tom-passives:CP_EIA-3216-12_Kemet-S" H 6938 1050 30  0001 C CNN
 F 3 "" H 6900 1200 60  0001 C CNN
 F 4 "478-12404-1-ND" H 6900 1200 50  0001 C CNN "Vendor"
@@
 Wire Wire Line
 	6900 1000 7100 1000
-Wire Wire Line
-	6650 1400 6900 1400
-Connection ~ 6900 1400
-Wire Wire Line
-	6900 1400 7100 1400
 $Comp
 L tom-passives:C C?
@@
 VCCO_34
 $Comp
-L tom-passives:C C?
+L tom-passives:CP_Small C?
 U 1 1 5E9F722D
 P 6900 2350
@@
 F 0 "C86" V 6850 1550 40  0000 L CNN
 F 1 "100uF/6.3V/X5R" V 6950 1550 40  0000 L CNN
-F 2 "tom-passives:C_1206_3216Metric" H 6938 2200 30  0001 C CNN
+F 2 "tom-passives:CP_EIA-3216-12_Kemet-S" H 6938 2200 30  0001 C CNN
 F 3 "" H 6900 2350 60  0001 C CNN
 F 4 "478-12404-1-ND" H 6900 2350 50  0001 C CNN "Vendor"
@@
 Wire Wire Line
 	6900 2150 7100 2150
-Wire Wire Line
-	6650 2550 6900 2550
-Connection ~ 6900 2550
-Wire Wire Line
-	6900 2550 7100 2550
 $Comp
 L tom-passives:C C?
@@
 ULX3S
 $Comp
-L tom-passives:C C?
+L tom-passives:CP_Small C?
 U 1 1 5EAAA6C6
 P 9750 3750
@@
 F 0 "C23" H 9650 4150 40  0000 L CNN
 F 1 "100uF/6.3V/X5R" H 9450 4050 40  0000 L CNN
-F 2 "tom-passives:C_1206_3216Metric" H 9788 3600 30  0001 C CNN
+F 2 "tom-passives:CP_EIA-3216-12_Kemet-S" H 9788 3600 30  0001 C CNN
 F 3 "" H 9750 3750 60  0001 C CNN
 F 4 "478-12404-1-ND" H 9750 3750 50  0001 C CNN "Vendor"
@@
 VCCO_35
 $Comp
-L tom-passives:C C?
+L tom-passives:CP_Small C?
 U 1 1 5EAE8169
 P 8200 5950
@@
 F 0 "C18" H 8350 6000 40  0000 L CNN
 F 1 "100uF/6.3V/X5R" H 8350 5900 40  0000 L CNN
-F 2 "tom-passives:C_1206_3216Metric" H 8238 5800 30  0001 C CNN
+F 2 "tom-passives:CP_EIA-3216-12_Kemet-S" H 8238 5800 30  0001 C CNN
 F 3 "" H 8200 5950 60  0001 C CNN
 F 4 "478-12404-1-ND" H 8200 5950 50  0001 C CNN "Vendor"
@@
 NoConn ~ 5300 3550
 NoConn ~ 5300 3650
+Wire Wire Line
+	6900 1000 6900 1100
+Wire Wire Line
+	6650 1400 6900 1400
+Wire Wire Line
+	6900 1300 6900 1400
+Connection ~ 6900 1400
+Wire Wire Line
+	6900 1400 7100 1400
+Wire Wire Line
+	6900 2150 6900 2250
+Wire Wire Line
+	6650 2550 6900 2550
+Wire Wire Line
+	6900 2450 6900 2550
+Connection ~ 6900 2550
+Wire Wire Line
+	6900 2550 7100 2550
+Wire Wire Line
+	9750 3550 9750 3650
+Wire Wire Line
+	9750 3850 9750 3950
+Wire Wire Line
+	8200 5750 8200 5850
+Wire Wire Line
+	8200 6050 8200 6150
 $EndSCHEMATC

Commit message: v2 hardware: Aug2020/rc2 version - flip tx/rx pairs on s2 - add lcsc part numbers
rc2 errata schematic
- change serial port connector to add +3.3V ? (8-pin)(NO)
- add test points for flash pre-programming
- smaller package on input direction diodes (NO)
- bom dupe errors
- remove all p/s 0R bringup parts
- optimise bom (use 1.5k for led, 10k/4.7k for i2c pullups)
- done led is bright (change to 4.7k)
- improve shield grounding with RC
- check actual values of RGB resistors
- remove caps from clock inputs

rc2 errata pcb
- no gnd marking on serial port connector pins
- change serial port connector to add +3.3V ? (8-pin) (NO)
- no test points for flash pre-programming
- missing caps on xtal? (No but select xtal carefully)
- Cfg sel pins on clock chip?
- No silk on test points
- No +/- pair numbering on silk
- vcc test points for clk pre-programming? (or use bootloader)
- random silk circle under S2
- smaller package on input direction diodes (NO)
- no polarity on 100uF tantalum
- some via in or close to pads
- wrong button package (change from feather to chinese)
- gnd/vcc labels swapped at high end of J2
- clock chip OUT0_SEL_I2CB needs to be tied high after programming
- check teardrops
- power diode footprint marking reverse
- LEDs use cap footprint
Parts:
- C18, C23, C85, C86: LCSC (none) -> C15008
- C87, C88, C89, C90: LCSC (none) -> C23733
- C91, C92, C93, C94, C95, C96, C97, C98: LCSC (none) -> C47339
- J1, TP1, TP2, TP3, TP4, U1: LCSC (none) -> DNP
Changed lines of the file:
@@
 F 2 "artix7-pcie-v2:Socket_Strip_Angled_2x20" H 8500 4750 50  0001 C CNN
 F 3 "~" H 8500 4750 50  0001 C CNN
+F 4 "DNP" H 8500 4750 50  0001 C CNN "LCSC"
 	1    8500 4750
 	-1   0    0    -1
@@
 F 2 "tom-mechanical:TestPoint_Pad_D1.5mm" H 6250 2350 50  0001 C CNN
 F 3 "~" H 6250 2350 50  0001 C CNN
+F 4 "DNP" H 6050 2350 50  0001 C CNN "LCSC"
 	1    6050 2350
 	0    1    -1   0
@@
 F 2 "tom-mechanical:TestPoint_Pad_D1.5mm" H 6250 2450 50  0001 C CNN
 F 3 "~" H 6250 2450 50  0001 C CNN
+F 4 "DNP" H 6050 2450 50  0001 C CNN "LCSC"
 	1    6050 2450
 	0    1    1    0
@@
 F 2 "tom-mechanical:TestPoint_Pad_D1.5mm" H 1050 3900 50  0001 C CNN
 F 3 "~" H 1050 3900 50  0001 C CNN
+F 4 "DNP" H 850 3900 50  0001 C CNN "LCSC"
 	1    850  3900
 	1    0    0    -1
@@
 F 2 "tom-mechanical:TestPoint_Pad_D1.5mm" H 800 3900 50  0001 C CNN
 F 3 "~" H 800 3900 50  0001 C CNN
+F 4 "DNP" H 600 3900 50  0001 C CNN "LCSC"
 	1    600  3900
 	1    0    0    -1
@@
 F 2 "artix7-pcie-v2:Xilinx_FGG484" H 3300 4150 50  0001 C CNN
 F 3 "" H 3300 4150 50  0000 C CNN
+F 4 "DNP" H 3300 4150 50  0001 C CNN "LCSC"
 	3    3300 4150
 	1    0    0    -1
@@
 F 3 "" H 6900 1200 60  0001 C CNN
 F 4 "478-12404-1-ND" H 6900 1200 50  0001 C CNN "Vendor"
+F 5 "C15008" H 6900 1200 50  0001 C CNN "LCSC"
 	1    6900 1200
 	1    0    0    -1
@@
 F 3 "" H 7100 1200 60  0001 C CNN
 F 4 "490-5915-1-ND" H 7100 1200 50  0001 C CNN "Vendor"
+F 5 "C23733" H 7100 1200 50  0001 C CNN "LCSC"
 	1    7100 1200
 	1    0    0    -1
@@
 F 3 "" H 7300 1200 60  0001 C CNN
 F 4 "490-5915-1-ND" H 7300 1200 50  0001 C CNN "Vendor"
+F 5 "C23733" H 7300 1200 50  0001 C CNN "LCSC"
 	1    7300 1200
 	1    0    0    -1
@@
 F 3 "" H 7500 1200 60  0001 C CNN
 F 4 "1276-CL05Y474KP5VPNCCT-ND" H 7500 1200 50  0001 C CNN "Vendor"
+F 5 "C47339" H 7500 1200 50  0001 C CNN "LCSC"
 	1    7500 1200
 	1    0    0    -1
@@
 F 3 "" H 7700 1200 60  0001 C CNN
 F 4 "1276-CL05Y474KP5VPNCCT-ND" H 7700 1200 50  0001 C CNN "Vendor"
+F 5 "C47339" H 7700 1200 50  0001 C CNN "LCSC"
 	1    7700 1200
 	1    0    0    -1
@@
 F 3 "" H 7900 1200 60  0001 C CNN
 F 4 "1276-CL05Y474KP5VPNCCT-ND" H 7900 1200 50  0001 C CNN "Vendor"
+F 5 "C47339" H 7900 1200 50  0001 C CNN "LCSC"
 	1    7900 1200
 	1    0    0    -1
@@
 F 3 "" H 8100 1200 60  0001 C CNN
 F 4 "1276-CL05Y474KP5VPNCCT-ND" H 8100 1200 50  0001 C CNN "Vendor"
+F 5 "C47339" H 8100 1200 50  0001 C CNN "LCSC"
 	1    8100 1200
 	1    0    0    -1
@@
 F 3 "" H 6900 2350 60  0001 C CNN
 F 4 "478-12404-1-ND" H 6900 2350 50  0001 C CNN "Vendor"
+F 5 "C15008" H 6900 2350 50  0001 C CNN "LCSC"
 	1    6900 2350
 	1    0    0    -1
@@
 F 3 "" H 7100 2350 60  0001 C CNN
 F 4 "490-5915-1-ND" H 7100 2350 50  0001 C CNN "Vendor"
+F 5 "C23733" H 7100 2350 50  0001 C CNN "LCSC"
 	1    7100 2350
 	1    0    0    -1
@@
 F 3 "" H 7300 2350 60  0001 C CNN
 F 4 "490-5915-1-ND" H 7300 2350 50  0001 C CNN "Vendor"
+F 5 "C23733" H 7300 2350 50  0001 C CNN "LCSC"
 	1    7300 2350
 	1    0    0    -1
@@
 F 3 "" H 7500 2350 60  0001 C CNN
 F 4 "1276-CL05Y474KP5VPNCCT-ND" H 7500 2350 50  0001 C CNN "Vendor"
+F 5 "C47339" H 7500 2350 50  0001 C CNN "LCSC"
 	1    7500 2350
 	1    0    0    -1
@@
 F 3 "" H 7700 2350 60  0001 C CNN
 F 4 "1276-CL05Y474KP5VPNCCT-ND" H 7700 2350 50  0001 C CNN "Vendor"
+F 5 "C47339" H 7700 2350 50  0001 C CNN "LCSC"
 	1    7700 2350
 	1    0    0    -1
@@
 F 3 "" H 7900 2350 60  0001 C CNN
 F 4 "1276-CL05Y474KP5VPNCCT-ND" H 7900 2350 50  0001 C CNN "Vendor"
+F 5 "C47339" H 7900 2350 50  0001 C CNN "LCSC"
 	1    7900 2350
 	1    0    0    -1
@@
 F 3 "" H 8100 2350 60  0001 C CNN
 F 4 "1276-CL05Y474KP5VPNCCT-ND" H 8100 2350 50  0001 C CNN "Vendor"
+F 5 "C47339" H 8100 2350 50  0001 C CNN "LCSC"
 	1    8100 2350
 	1    0    0    -1
@@
 F 3 "" H 9750 3750 60  0001 C CNN
 F 4 "478-12404-1-ND" H 9750 3750 50  0001 C CNN "Vendor"
+F 5 "C15008" H 9750 3750 50  0001 C CNN "LCSC"
 	1    9750 3750
 	1    0    0    -1
@@
 F 3 "" H 8200 5950 60  0001 C CNN
 F 4 "478-12404-1-ND" H 8200 5950 50  0001 C CNN "Vendor"
+F 5 "C15008" H 8200 5950 50  0001 C CNN "LCSC"
 	1    8200 5950
 	1    0    0    -1

Commit message: v2 hardware: change 100uF to 3528 for jlcpcb
Parts:
- C18, C23, C85, C86: footprint tom-passives:CP_EIA-3216-12_Kemet-S -> tom-passives:CP_EIA-3528-15_AVX-H
Changed lines of the file:
@@
 F 0 "C85" V 6850 400 40  0000 L CNN
 F 1 "100uF/6.3V/X5R" V 6950 400 40  0000 L CNN
-F 2 "tom-passives:CP_EIA-3216-12_Kemet-S" H 6938 1050 30  0001 C CNN
+F 2 "tom-passives:CP_EIA-3528-15_AVX-H" H 6938 1050 30  0001 C CNN
 F 3 "" H 6900 1200 60  0001 C CNN
 F 4 "478-12404-1-ND" H 6900 1200 50  0001 C CNN "Vendor"
@@
 F 0 "C86" V 6850 1550 40  0000 L CNN
 F 1 "100uF/6.3V/X5R" V 6950 1550 40  0000 L CNN
-F 2 "tom-passives:CP_EIA-3216-12_Kemet-S" H 6938 2200 30  0001 C CNN
+F 2 "tom-passives:CP_EIA-3528-15_AVX-H" H 6938 2200 30  0001 C CNN
 F 3 "" H 6900 2350 60  0001 C CNN
 F 4 "478-12404-1-ND" H 6900 2350 50  0001 C CNN "Vendor"
@@
 F 0 "C23" H 9650 4150 40  0000 L CNN
 F 1 "100uF/6.3V/X5R" H 9450 4050 40  0000 L CNN
-F 2 "tom-passives:CP_EIA-3216-12_Kemet-S" H 9788 3600 30  0001 C CNN
+F 2 "tom-passives:CP_EIA-3528-15_AVX-H" H 9788 3600 30  0001 C CNN
 F 3 "" H 9750 3750 60  0001 C CNN
 F 4 "478-12404-1-ND" H 9750 3750 50  0001 C CNN "Vendor"
@@
 F 0 "C18" H 8350 6000 40  0000 L CNN
 F 1 "100uF/6.3V/X5R" H 8350 5900 40  0000 L CNN
-F 2 "tom-passives:CP_EIA-3216-12_Kemet-S" H 8238 5800 30  0001 C CNN
+F 2 "tom-passives:CP_EIA-3528-15_AVX-H" H 8238 5800 30  0001 C CNN
 F 3 "" H 8200 5950 60  0001 C CNN
 F 4 "478-12404-1-ND" H 8200 5950 50  0001 C CNN "Vendor"

Commit message: v2 hardware: sep2020 run - fixed issues with parts missing from centroid file
Parts:
- C18, C23, C85, C86: LCSC C15008 -> C16133
Changed lines of the file:
@@
 F 3 "" H 6900 1200 60  0001 C CNN
 F 4 "478-12404-1-ND" H 6900 1200 50  0001 C CNN "Vendor"
-F 5 "C15008" H 6900 1200 50  0001 C CNN "LCSC"
+F 5 "C16133" H 6900 1200 50  0001 C CNN "LCSC"
 	1    6900 1200
 	1    0    0    -1
@@
 F 3 "" H 6900 2350 60  0001 C CNN
 F 4 "478-12404-1-ND" H 6900 2350 50  0001 C CNN "Vendor"
-F 5 "C15008" H 6900 2350 50  0001 C CNN "LCSC"
+F 5 "C16133" H 6900 2350 50  0001 C CNN "LCSC"
 	1    6900 2350
 	1    0    0    -1
@@
 F 3 "" H 9750 3750 60  0001 C CNN
 F 4 "478-12404-1-ND" H 9750 3750 50  0001 C CNN "Vendor"
-F 5 "C15008" H 9750 3750 50  0001 C CNN "LCSC"
+F 5 "C16133" H 9750 3750 50  0001 C CNN "LCSC"
 	1    9750 3750
 	1    0    0    -1
@@
 F 3 "" H 8200 5950 60  0001 C CNN
 F 4 "478-12404-1-ND" H 8200 5950 50  0001 C CNN "Vendor"
-F 5 "C15008" H 8200 5950 50  0001 C CNN "LCSC"
+F 5 "C16133" H 8200 5950 50  0001 C CNN "LCSC"
 	1    8200 5950
 	1    0    0    -1
