File: hardware/v2/artix7-pcie-v2-power-fpga.sch (KiCad schematic (older format))
At the start: 1 part, among them U1 XC7A75T-FGG484

Commit message: v2 pcb/schematic update : drc passing, need to add caps
Connections:
- net VCCINT: now also U1.T10 (VCCINT)
Changed lines of the file:
@@
 EESchema Schematic File Version 4
-LIBS:artix7-pcie-v2-cache
 EELAYER 30 0
 EELAYER END
 $Descr A4 11693 8268
 encoding utf-8
-Sheet 3 7
+Sheet 7 7
 Title ""
 Date ""
@@
 	1350 1700 1350 1800
 Wire Wire Line
-	3350 2650 3350 2600
+	3350 2700 3350 2600
 Connection ~ 3350 1400
 Wire Wire Line

Commit message: v2 hardware: pcb progress commit, 155 unrouted
Parts:
- added C42, C44: 100uF/6.3V/X5R, tom-passives:C_1206_3216Metric, symbol tom-passives:C
- added C43, C45, C46, C50, C70, C71, C72, C73: 4.7uF/6.3V/X5R, tom-passives:C_0402_1005Metric, symbol tom-passives:C
- added C49, C51, C52, C53, C54, C55, C56, C58, C59, C69, C74, C75, C76, C77: 0.47uF/6.3V/X5R, tom-passives:C_0402_1005Metric, symbol tom-passives:C
Connections:
- net GND: now also C42.2, C43.2, C44.2, C45.2, C46.2, C49.2, C50.2, C51.2, C52.2, C53.2, C54.2, C55.2, C56.2, C58.2, C59.2, C69.2, C70.2, C71.2, C72.2, C73.2, C74.2, C75.2, C76.2, C77.2
- net VCCAUX: now also C42.1, C45.1, C50.1, C51.1, C52.1, C54.1, C56.1, C70.1, C74.1
- net VCCBRAM: now also C43.1, C49.1, C69.1
- net VCCINT: now also C44.1, C46.1, C53.1, C55.1, C58.1, C59.1, C71.1, C72.1, C73.1, C75.1, C76.1, C77.1

Commit message: v2 hardware: add Digikey part numbers to schematic and generate bom
Parts:
- C42, C44: Vendor (none) -> 478-12404-1-ND
- C43, C45, C46, C50, C70, C71, C72, C73: Vendor (none) -> 490-5915-1-ND
- C49, C51, C52, C53, C54, C55, C56, C58, C59, C69, C74, C75, C76, C77: Vendor (none) -> 1276-CL05Y474KP5VPNCCT-ND
Changed lines of the file:
@@
 F 2 "tom-passives:C_1206_3216Metric" H 6338 1900 30  0001 C CNN
 F 3 "" H 6300 2050 60  0001 C CNN
+F 4 "478-12404-1-ND" H 6300 2050 50  0001 C CNN "Vendor"
 	1    6300 2050
 	1    0    0    -1
@@
 F 2 "tom-passives:C_0402_1005Metric" H 6538 1900 30  0001 C CNN
 F 3 "" H 6500 2050 60  0001 C CNN
+F 4 "490-5915-1-ND" H 6500 2050 50  0001 C CNN "Vendor"
 	1    6500 2050
 	1    0    0    -1
@@
 F 2 "tom-passives:C_0402_1005Metric" H 6338 3050 30  0001 C CNN
 F 3 "" H 6300 3200 60  0001 C CNN
+F 4 "490-5915-1-ND" H 6300 3200 50  0001 C CNN "Vendor"
 	1    6300 3200
 	1    0    0    -1
@@
 F 2 "tom-passives:C_1206_3216Metric" H 6338 4200 30  0001 C CNN
 F 3 "" H 6300 4350 60  0001 C CNN
+F 4 "478-12404-1-ND" H 6300 4350 50  0001 C CNN "Vendor"
 	1    6300 4350
 	1    0    0    -1
@@
 F 2 "tom-passives:C_0402_1005Metric" H 6538 4200 30  0001 C CNN
 F 3 "" H 6500 4350 60  0001 C CNN
+F 4 "490-5915-1-ND" H 6500 4350 50  0001 C CNN "Vendor"
 	1    6500 4350
 	1    0    0    -1
@@
 F 2 "tom-passives:C_0402_1005Metric" H 6738 1900 30  0001 C CNN
 F 3 "" H 6700 2050 60  0001 C CNN
+F 4 "490-5915-1-ND" H 6700 2050 50  0001 C CNN "Vendor"
 	1    6700 2050
 	1    0    0    -1
@@
 F 2 "tom-passives:C_0402_1005Metric" H 7138 1900 30  0001 C CNN
 F 3 "" H 7100 2050 60  0001 C CNN
+F 4 "1276-CL05Y474KP5VPNCCT-ND" H 7100 2050 50  0001 C CNN "Vendor"
 	1    7100 2050
 	1    0    0    -1
@@
 F 2 "tom-passives:C_0402_1005Metric" H 7338 1900 30  0001 C CNN
 F 3 "" H 7300 2050 60  0001 C CNN
+F 4 "1276-CL05Y474KP5VPNCCT-ND" H 7300 2050 50  0001 C CNN "Vendor"
 	1    7300 2050
 	1    0    0    -1
@@
 F 2 "tom-passives:C_0402_1005Metric" H 7538 1900 30  0001 C CNN
 F 3 "" H 7500 2050 60  0001 C CNN
+F 4 "1276-CL05Y474KP5VPNCCT-ND" H 7500 2050 50  0001 C CNN "Vendor"
 	1    7500 2050
 	1    0    0    -1
@@
 F 2 "tom-passives:C_0402_1005Metric" H 7738 1900 30  0001 C CNN
 F 3 "" H 7700 2050 60  0001 C CNN
+F 4 "1276-CL05Y474KP5VPNCCT-ND" H 7700 2050 50  0001 C CNN "Vendor"
 	1    7700 2050
 	1    0    0    -1
@@
 F 2 "tom-passives:C_0402_1005Metric" H 6538 3050 30  0001 C CNN
 F 3 "" H 6500 3200 60  0001 C CNN
+F 4 "1276-CL05Y474KP5VPNCCT-ND" H 6500 3200 50  0001 C CNN "Vendor"
 	1    6500 3200
 	1    0    0    -1
@@
 F 2 "tom-passives:C_0402_1005Metric" H 7338 4200 30  0001 C CNN
 F 3 "" H 7300 4350 60  0001 C CNN
+F 4 "1276-CL05Y474KP5VPNCCT-ND" H 7300 4350 50  0001 C CNN "Vendor"
 	1    7300 4350
 	1    0    0    -1
@@
 F 2 "tom-passives:C_0402_1005Metric" H 7538 4200 30  0001 C CNN
 F 3 "" H 7500 4350 60  0001 C CNN
+F 4 "1276-CL05Y474KP5VPNCCT-ND" H 7500 4350 50  0001 C CNN "Vendor"
 	1    7500 4350
 	1    0    0    -1
@@
 F 2 "tom-passives:C_0402_1005Metric" H 7738 4200 30  0001 C CNN
 F 3 "" H 7700 4350 60  0001 C CNN
+F 4 "1276-CL05Y474KP5VPNCCT-ND" H 7700 4350 50  0001 C CNN "Vendor"
 	1    7700 4350
 	1    0    0    -1
@@
 F 2 "tom-passives:C_0402_1005Metric" H 7938 4200 30  0001 C CNN
 F 3 "" H 7900 4350 60  0001 C CNN
+F 4 "1276-CL05Y474KP5VPNCCT-ND" H 7900 4350 50  0001 C CNN "Vendor"
 	1    7900 4350
 	1    0    0    -1
@@
 F 2 "tom-passives:C_0402_1005Metric" H 6738 4200 30  0001 C CNN
 F 3 "" H 6700 4350 60  0001 C CNN
+F 4 "490-5915-1-ND" H 6700 4350 50  0001 C CNN "Vendor"
 	1    6700 4350
 	1    0    0    -1
@@
 F 2 "tom-passives:C_0402_1005Metric" H 6938 4200 30  0001 C CNN
 F 3 "" H 6900 4350 60  0001 C CNN
+F 4 "490-5915-1-ND" H 6900 4350 50  0001 C CNN "Vendor"
 	1    6900 4350
 	1    0    0    -1
@@
 F 2 "tom-passives:C_0402_1005Metric" H 7138 4200 30  0001 C CNN
 F 3 "" H 7100 4350 60  0001 C CNN
+F 4 "490-5915-1-ND" H 7100 4350 50  0001 C CNN "Vendor"
 	1    7100 4350
 	1    0    0    -1
@@
 F 2 "tom-passives:C_0402_1005Metric" H 8138 4200 30  0001 C CNN
 F 3 "" H 8100 4350 60  0001 C CNN
+F 4 "1276-CL05Y474KP5VPNCCT-ND" H 8100 4350 50  0001 C CNN "Vendor"
 	1    8100 4350
 	1    0    0    -1
@@
 F 2 "tom-passives:C_0402_1005Metric" H 8338 4200 30  0001 C CNN
 F 3 "" H 8300 4350 60  0001 C CNN
+F 4 "1276-CL05Y474KP5VPNCCT-ND" H 8300 4350 50  0001 C CNN "Vendor"
 	1    8300 4350
 	1    0    0    -1
@@
 F 2 "tom-passives:C_0402_1005Metric" H 8538 4200 30  0001 C CNN
 F 3 "" H 8500 4350 60  0001 C CNN
+F 4 "1276-CL05Y474KP5VPNCCT-ND" H 8500 4350 50  0001 C CNN "Vendor"
 	1    8500 4350
 	1    0    0    -1
@@
 F 2 "tom-passives:C_0402_1005Metric" H 6738 3050 30  0001 C CNN
 F 3 "" H 6700 3200 60  0001 C CNN
+F 4 "1276-CL05Y474KP5VPNCCT-ND" H 6700 3200 50  0001 C CNN "Vendor"
 	1    6700 3200
 	1    0    0    -1
@@
 F 2 "tom-passives:C_0402_1005Metric" H 6938 1900 30  0001 C CNN
 F 3 "" H 6900 2050 60  0001 C CNN
+F 4 "490-5915-1-ND" H 6900 2050 50  0001 C CNN "Vendor"
 	1    6900 2050
 	1    0    0    -1
@@
 F 2 "tom-passives:C_0402_1005Metric" H 7938 1900 30  0001 C CNN
 F 3 "" H 7900 2050 60  0001 C CNN
+F 4 "1276-CL05Y474KP5VPNCCT-ND" H 7900 2050 50  0001 C CNN "Vendor"
 	1    7900 2050
 	1    0    0    -1

Commit message: v2 hardware: aug2020 pcb updates
Parts:
- C42, C44: footprint tom-passives:C_1206_3216Metric -> tom-passives:CP_EIA-3216-12_Kemet-S; symbol tom-passives:C -> tom-passives:CP_Small
Changed lines of the file:
@@
 	1200 2100 1200 1400
 $Comp
-L tom-passives:C C?
+L tom-passives:CP_Small C?
 U 1 1 5E7EC0F9
 P 6300 2050
@@
 F 0 "C42" V 6250 1250 40  0000 L CNN
 F 1 "100uF/6.3V/X5R" V 6350 1250 40  0000 L CNN
-F 2 "tom-passives:C_1206_3216Metric" H 6338 1900 30  0001 C CNN
+F 2 "tom-passives:CP_EIA-3216-12_Kemet-S" H 6338 1900 30  0001 C CNN
 F 3 "" H 6300 2050 60  0001 C CNN
 F 4 "478-12404-1-ND" H 6300 2050 50  0001 C CNN "Vendor"
@@
 Wire Wire Line
 	6300 1850 6500 1850
-Wire Wire Line
-	6050 2250 6300 2250
-Connection ~ 6300 2250
-Wire Wire Line
-	6300 2250 6500 2250
 $Comp
 L tom-passives:C C?
@@
 	6050 3000 6300 3000
 $Comp
-L tom-passives:C C?
+L tom-passives:CP_Small C?
 U 1 1 5E829A46
 P 6300 4350
@@
 F 0 "C44" V 6250 3550 40  0000 L CNN
 F 1 "100uF/6.3V/X5R" V 6350 3550 40  0000 L CNN
-F 2 "tom-passives:C_1206_3216Metric" H 6338 4200 30  0001 C CNN
+F 2 "tom-passives:CP_EIA-3216-12_Kemet-S" H 6338 4200 30  0001 C CNN
 F 3 "" H 6300 4350 60  0001 C CNN
 F 4 "478-12404-1-ND" H 6300 4350 50  0001 C CNN "Vendor"
@@
 	1    0    0    -1
 $EndComp
-Wire Wire Line
-	6300 4550 6100 4550
 Wire Wire Line
 	6300 4150 6100 4150
@@
 Connection ~ 6300 4150
 Connection ~ 6500 4150
-Connection ~ 6300 4550
 Connection ~ 6500 4550
-Wire Wire Line
-	6500 4550 6300 4550
 $Comp
 L tom-passives:C C?
@@
 Wire Wire Line
 	6500 4550 6700 4550
+Wire Wire Line
+	6300 1950 6300 1850
+Wire Wire Line
+	6050 2250 6300 2250
+Wire Wire Line
+	6300 2150 6300 2250
+Connection ~ 6300 2250
+Wire Wire Line
+	6300 2250 6500 2250
+Wire Wire Line
+	6300 4150 6300 4250
+Wire Wire Line
+	6100 4550 6300 4550
+Wire Wire Line
+	6300 4450 6300 4550
+Connection ~ 6300 4550
+Wire Wire Line
+	6300 4550 6500 4550
 $EndSCHEMATC

Commit message: v2 hardware: Aug2020/rc2 version - flip tx/rx pairs on s2 - add lcsc part numbers
rc2 errata schematic
- change serial port connector to add +3.3V ? (8-pin)(NO)
- add test points for flash pre-programming
- smaller package on input direction diodes (NO)
- bom dupe errors
- remove all p/s 0R bringup parts
- optimise bom (use 1.5k for led, 10k/4.7k for i2c pullups)
- done led is bright (change to 4.7k)
- improve shield grounding with RC
- check actual values of RGB resistors
- remove caps from clock inputs

rc2 errata pcb
- no gnd marking on serial port connector pins
- change serial port connector to add +3.3V ? (8-pin) (NO)
- no test points for flash pre-programming
- missing caps on xtal? (No but select xtal carefully)
- Cfg sel pins on clock chip?
- No silk on test points
- No +/- pair numbering on silk
- vcc test points for clk pre-programming? (or use bootloader)
- random silk circle under S2
- smaller package on input direction diodes (NO)
- no polarity on 100uF tantalum
- some via in or close to pads
- wrong button package (change from feather to chinese)
- gnd/vcc labels swapped at high end of J2
- clock chip OUT0_SEL_I2CB needs to be tied high after programming
- check teardrops
- power diode footprint marking reverse
- LEDs use cap footprint
Parts:
- C42, C44: LCSC (none) -> C15008
- C43, C45, C46, C50, C70, C71, C72, C73: LCSC (none) -> C23733
- C49, C51, C52, C53, C54, C55, C56, C58, C59, C69, C74, C75, C76, C77: LCSC (none) -> C47339
- U1: LCSC (none) -> DNP
Changed lines of the file:
@@
 F 2 "artix7-pcie-v2:Xilinx_FGG484" H 2350 4300 50  0001 C CNN
 F 3 "" H 2350 4300 50  0000 C CNN
+F 4 "DNP" H 2350 4300 50  0001 C CNN "LCSC"
 	7    2350 4300
 	1    0    0    -1
@@
 F 3 "" H 6300 2050 60  0001 C CNN
 F 4 "478-12404-1-ND" H 6300 2050 50  0001 C CNN "Vendor"
+F 5 "C15008" H 6300 2050 50  0001 C CNN "LCSC"
 	1    6300 2050
 	1    0    0    -1
@@
 F 3 "" H 6500 2050 60  0001 C CNN
 F 4 "490-5915-1-ND" H 6500 2050 50  0001 C CNN "Vendor"
+F 5 "C23733" H 6500 2050 50  0001 C CNN "LCSC"
 	1    6500 2050
 	1    0    0    -1
@@
 F 3 "" H 6300 3200 60  0001 C CNN
 F 4 "490-5915-1-ND" H 6300 3200 50  0001 C CNN "Vendor"
+F 5 "C23733" H 6300 3200 50  0001 C CNN "LCSC"
 	1    6300 3200
 	1    0    0    -1
@@
 F 3 "" H 6300 4350 60  0001 C CNN
 F 4 "478-12404-1-ND" H 6300 4350 50  0001 C CNN "Vendor"
+F 5 "C15008" H 6300 4350 50  0001 C CNN "LCSC"
 	1    6300 4350
 	1    0    0    -1
@@
 F 3 "" H 6500 4350 60  0001 C CNN
 F 4 "490-5915-1-ND" H 6500 4350 50  0001 C CNN "Vendor"
+F 5 "C23733" H 6500 4350 50  0001 C CNN "LCSC"
 	1    6500 4350
 	1    0    0    -1
@@
 F 3 "" H 6700 2050 60  0001 C CNN
 F 4 "490-5915-1-ND" H 6700 2050 50  0001 C CNN "Vendor"
+F 5 "C23733" H 6700 2050 50  0001 C CNN "LCSC"
 	1    6700 2050
 	1    0    0    -1
@@
 F 3 "" H 7100 2050 60  0001 C CNN
 F 4 "1276-CL05Y474KP5VPNCCT-ND" H 7100 2050 50  0001 C CNN "Vendor"
+F 5 "C47339" H 7100 2050 50  0001 C CNN "LCSC"
 	1    7100 2050
 	1    0    0    -1
@@
 F 3 "" H 7300 2050 60  0001 C CNN
 F 4 "1276-CL05Y474KP5VPNCCT-ND" H 7300 2050 50  0001 C CNN "Vendor"
+F 5 "C47339" H 7300 2050 50  0001 C CNN "LCSC"
 	1    7300 2050
 	1    0    0    -1
@@
 F 3 "" H 7500 2050 60  0001 C CNN
 F 4 "1276-CL05Y474KP5VPNCCT-ND" H 7500 2050 50  0001 C CNN "Vendor"
+F 5 "C47339" H 7500 2050 50  0001 C CNN "LCSC"
 	1    7500 2050
 	1    0    0    -1
@@
 F 3 "" H 7700 2050 60  0001 C CNN
 F 4 "1276-CL05Y474KP5VPNCCT-ND" H 7700 2050 50  0001 C CNN "Vendor"
+F 5 "C47339" H 7700 2050 50  0001 C CNN "LCSC"
 	1    7700 2050
 	1    0    0    -1
@@
 F 3 "" H 6500 3200 60  0001 C CNN
 F 4 "1276-CL05Y474KP5VPNCCT-ND" H 6500 3200 50  0001 C CNN "Vendor"
+F 5 "C47339" H 6500 3200 50  0001 C CNN "LCSC"
 	1    6500 3200
 	1    0    0    -1
@@
 F 3 "" H 7300 4350 60  0001 C CNN
 F 4 "1276-CL05Y474KP5VPNCCT-ND" H 7300 4350 50  0001 C CNN "Vendor"
+F 5 "C47339" H 7300 4350 50  0001 C CNN "LCSC"
 	1    7300 4350
 	1    0    0    -1
@@
 F 3 "" H 7500 4350 60  0001 C CNN
 F 4 "1276-CL05Y474KP5VPNCCT-ND" H 7500 4350 50  0001 C CNN "Vendor"
+F 5 "C47339" H 7500 4350 50  0001 C CNN "LCSC"
 	1    7500 4350
 	1    0    0    -1
@@
 F 3 "" H 7700 4350 60  0001 C CNN
 F 4 "1276-CL05Y474KP5VPNCCT-ND" H 7700 4350 50  0001 C CNN "Vendor"
+F 5 "C47339" H 7700 4350 50  0001 C CNN "LCSC"
 	1    7700 4350
 	1    0    0    -1
@@
 F 3 "" H 7900 4350 60  0001 C CNN
 F 4 "1276-CL05Y474KP5VPNCCT-ND" H 7900 4350 50  0001 C CNN "Vendor"
+F 5 "C47339" H 7900 4350 50  0001 C CNN "LCSC"
 	1    7900 4350
 	1    0    0    -1
@@
 F 3 "" H 6700 4350 60  0001 C CNN
 F 4 "490-5915-1-ND" H 6700 4350 50  0001 C CNN "Vendor"
+F 5 "C23733" H 6700 4350 50  0001 C CNN "LCSC"
 	1    6700 4350
 	1    0    0    -1
@@
 F 3 "" H 6900 4350 60  0001 C CNN
 F 4 "490-5915-1-ND" H 6900 4350 50  0001 C CNN "Vendor"
+F 5 "C23733" H 6900 4350 50  0001 C CNN "LCSC"
 	1    6900 4350
 	1    0    0    -1
@@
 F 3 "" H 7100 4350 60  0001 C CNN
 F 4 "490-5915-1-ND" H 7100 4350 50  0001 C CNN "Vendor"
+F 5 "C23733" H 7100 4350 50  0001 C CNN "LCSC"
 	1    7100 4350
 	1    0    0    -1
@@
 F 3 "" H 8100 4350 60  0001 C CNN
 F 4 "1276-CL05Y474KP5VPNCCT-ND" H 8100 4350 50  0001 C CNN "Vendor"
+F 5 "C47339" H 8100 4350 50  0001 C CNN "LCSC"
 	1    8100 4350
 	1    0    0    -1
@@
 F 3 "" H 8300 4350 60  0001 C CNN
 F 4 "1276-CL05Y474KP5VPNCCT-ND" H 8300 4350 50  0001 C CNN "Vendor"
+F 5 "C47339" H 8300 4350 50  0001 C CNN "LCSC"
 	1    8300 4350
 	1    0    0    -1
@@
 F 3 "" H 8500 4350 60  0001 C CNN
 F 4 "1276-CL05Y474KP5VPNCCT-ND" H 8500 4350 50  0001 C CNN "Vendor"
+F 5 "C47339" H 8500 4350 50  0001 C CNN "LCSC"
 	1    8500 4350
 	1    0    0    -1
@@
 F 3 "" H 6700 3200 60  0001 C CNN
 F 4 "1276-CL05Y474KP5VPNCCT-ND" H 6700 3200 50  0001 C CNN "Vendor"
+F 5 "C47339" H 6700 3200 50  0001 C CNN "LCSC"
 	1    6700 3200
 	1    0    0    -1
@@
 F 3 "" H 6900 2050 60  0001 C CNN
 F 4 "490-5915-1-ND" H 6900 2050 50  0001 C CNN "Vendor"
+F 5 "C23733" H 6900 2050 50  0001 C CNN "LCSC"
 	1    6900 2050
 	1    0    0    -1
@@
 F 3 "" H 7900 2050 60  0001 C CNN
 F 4 "1276-CL05Y474KP5VPNCCT-ND" H 7900 2050 50  0001 C CNN "Vendor"
+F 5 "C47339" H 7900 2050 50  0001 C CNN "LCSC"
 	1    7900 2050
 	1    0    0    -1

Commit message: v2 hardware: change 100uF to 3528 for jlcpcb
Parts:
- C42, C44: footprint tom-passives:CP_EIA-3216-12_Kemet-S -> tom-passives:CP_EIA-3528-15_AVX-H
Changed lines of the file:
@@
 F 0 "C42" V 6250 1250 40  0000 L CNN
 F 1 "100uF/6.3V/X5R" V 6350 1250 40  0000 L CNN
-F 2 "tom-passives:CP_EIA-3216-12_Kemet-S" H 6338 1900 30  0001 C CNN
+F 2 "tom-passives:CP_EIA-3528-15_AVX-H" H 6338 1900 30  0001 C CNN
 F 3 "" H 6300 2050 60  0001 C CNN
 F 4 "478-12404-1-ND" H 6300 2050 50  0001 C CNN "Vendor"
@@
 F 0 "C44" V 6250 3550 40  0000 L CNN
 F 1 "100uF/6.3V/X5R" V 6350 3550 40  0000 L CNN
-F 2 "tom-passives:CP_EIA-3216-12_Kemet-S" H 6338 4200 30  0001 C CNN
+F 2 "tom-passives:CP_EIA-3528-15_AVX-H" H 6338 4200 30  0001 C CNN
 F 3 "" H 6300 4350 60  0001 C CNN
 F 4 "478-12404-1-ND" H 6300 4350 50  0001 C CNN "Vendor"

Commit message: v2 hardware: sep2020 run - fixed issues with parts missing from centroid file
Parts:
- C42, C44: LCSC C15008 -> C16133
Changed lines of the file:
@@
 F 3 "" H 6300 2050 60  0001 C CNN
 F 4 "478-12404-1-ND" H 6300 2050 50  0001 C CNN "Vendor"
-F 5 "C15008" H 6300 2050 50  0001 C CNN "LCSC"
+F 5 "C16133" H 6300 2050 50  0001 C CNN "LCSC"
 	1    6300 2050
 	1    0    0    -1
@@
 F 3 "" H 6300 4350 60  0001 C CNN
 F 4 "478-12404-1-ND" H 6300 4350 50  0001 C CNN "Vendor"
-F 5 "C15008" H 6300 4350 50  0001 C CNN "LCSC"
+F 5 "C16133" H 6300 4350 50  0001 C CNN "LCSC"
 	1    6300 4350
 	1    0    0    -1
