File: hardware/v2/artix7-pcie-v2.sch (KiCad schematic (older format))
At the start: 51 parts, among them J10 USB_B_Micro, J3 JTAG_EN, J6 JTAG, J7 Conn_01x02, J8 SER, SW1 PROG, SW2 USER, U1 XC7A75T-FGG484, U2 MX25L51245GZ2I-10G, U4 5P49V6965A000NLGI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

Commit message: v2 hardware: aug2020 pcb updates
Parts:
- removed C3, C4, C40, C41: 0.1uF/6.3V/X5R/PCIE, tom-passives:C_0402_1005Metric, symbol tom-passives:C
- added TP16, TP17, TP18, TP19, TP20: TestPoint, tom-mechanical:TestPoint_Pad_D1.5mm, symbol tom-mechanical:TestPoint
- R1, R51: value 1K/5% -> 4.7k/5%
- R10, R9: value 10K/5% -> 4.7k/5%
- R30, R4: value 1k/5% -> 1k/1%
- SW1, SW2: footprint tom-mechanical:SW_Push_1P1T_NO_CK_KMR2 -> tom-mechanical:SW_Push_1P1T_NO_Vertical_Wuerth_434133025816
Connections:
- net OUT2_N is gone; now on net CLKIN_N: U4.16 (OUT2B)
- net OUT2_P is gone; now on net CLKIN_P: U4.17 (OUT2)
- net OUT3_N is gone; now on net artix7-pcie-v2-serdes/MGT_REFCLK0_N: U4.13 (OUT3B)
- net OUT3_P is gone; now on net artix7-pcie-v2-serdes/MGT_REFCLK0_P: U4.14 (OUT3)
- net CFG_FLASH_CS: now also TP20.1
- net CFG_FLASH_MISO_D1: now also TP19.1
- net CFG_FLASH_MOSI_D0: now also TP18.1
- net SPI_FLASH_CLK: now also TP17.1
- net VCC: now also TP16.1
Changed lines of the file:
@@
 	7800 1500 7800 1800
 Wire Wire Line
-	7800 1800 5800 1800
-Wire Wire Line
-	5800 1800 5800 1900
-Wire Wire Line
-	5800 1900 3450 1900
+	7800 1800 5700 1800
+Wire Wire Line
+	5700 1800 5700 1900
+Wire Wire Line
+	5700 1900 3450 1900
 Wire Wire Line
 	7700 1600 8250 1600
 Text Label 8550 1100 0    50   ~ 0
 CFG_FLASH_MOSI_D0
-Wire Wire Line
-	7900 1400 9350 1400
 Connection ~ 7900 1400
 Wire Wire Line
 	8250 1600 8250 1100
 Wire Wire Line
-	8250 1100 9350 1100
-Wire Wire Line
 	6250 1400 6250 1900
 Wire Wire Line
@@
 Wire Wire Line
 	8350 1900 8350 1200
-Wire Wire Line
-	8350 1200 9350 1200
-Wire Wire Line
-	9350 1300 8450 1300
 Wire Wire Line
 	8450 1300 8450 2000
@@
 	6150 1500 6400 1500
 Wire Wire Line
-	9350 1500 8550 1500
+	9350 1500 8750 1500
 Wire Wire Line
 	8550 1500 8550 2100
@@
 P 4150 2850
 F 0 "R1" H 4221 2888 40  0000 L CNN
-F 1 "1K/5%" H 4221 2812 40  0000 L CNN
+F 1 "4.7k/5%" H 4221 2812 40  0000 L CNN
 F 2 "tom-passives:R_0402_1005Metric" V 4080 2850 30  0001 C CNN
 F 3 "" H 4150 2850 30  0000 C CNN
@@
 P 5850 2450
 F 0 "R4" H 5921 2488 40  0000 L CNN
-F 1 "1k/5%" H 5921 2412 40  0000 L CNN
+F 1 "1k/1%" H 5921 2412 40  0000 L CNN
 F 2 "tom-passives:R_0402_1005Metric" V 5780 2450 30  0001 C CNN
 F 3 "" H 5850 2450 30  0000 C CNN
@@
 F 0 "SW1" H 5450 3535 50  0000 C CNN
 F 1 "PROG" H 5450 3444 50  0000 C CNN
-F 2 "tom-mechanical:SW_Push_1P1T_NO_CK_KMR2" H 5450 3300 50  0001 C CNN
+F 2 "tom-mechanical:SW_Push_1P1T_NO_Vertical_Wuerth_434133025816" H 5450 3300 50  0001 C CNN
 F 3 "~" H 5450 3300 50  0001 C CNN
 	1    5450 3300
@@
 F 0 "SW2" H 8950 2035 50  0000 C CNN
 F 1 "USER" H 8950 1944 50  0000 C CNN
-F 2 "tom-mechanical:SW_Push_1P1T_NO_CK_KMR2" H 8950 1800 50  0001 C CNN
+F 2 "tom-mechanical:SW_Push_1P1T_NO_Vertical_Wuerth_434133025816" H 8950 1800 50  0001 C CNN
 F 3 "~" H 8950 1800 50  0001 C CNN
 	1    8950 1800
@@
 P 8950 2500
 F 0 "R30" V 8765 2500 40  0000 C CNN
-F 1 "1k/5%" V 8841 2500 40  0000 C CNN
+F 1 "1k/1%" V 8841 2500 40  0000 C CNN
 F 2 "tom-passives:R_0402_1005Metric" V 8880 2500 30  0001 C CNN
 F 3 "" H 8950 2500 30  0000 C CNN
@@
 	1    0    0    -1
 $EndComp
-$Comp
-L tom-passives:C C?
-U 1 1 5E96B2FA
-P 3200 6600
-AR Path="/5E98B37D/5E96B2FA" Ref="C?"  Part="1"
-AR Path="/5E96B2FA" Ref="C3"  Part="1"
-F 0 "C3" V 2971 6600 40  0000 C CNN
-F 1 "0.1uF/6.3V/X5R/PCIE" V 3047 6600 40  0000 C CNN
-F 2 "tom-passives:C_0402_1005Metric" H 3238 6450 30  0001 C CNN
-F 3 "" H 3200 6600 60  0001 C CNN
-	1    3200 6600
-	0    -1   -1   0
-$EndComp
-$Comp
-L tom-passives:C C?
-U 1 1 5E9713AB
-P 3550 6700
-AR Path="/5E98B37D/5E9713AB" Ref="C?"  Part="1"
-AR Path="/5E9713AB" Ref="C4"  Part="1"
-F 0 "C4" V 3321 6700 40  0000 C CNN
-F 1 "0.1uF/6.3V/X5R/PCIE" V 3397 6700 40  0000 C CNN
-F 2 "tom-passives:C_0402_1005Metric" H 3588 6550 30  0001 C CNN
-F 3 "" H 3550 6700 60  0001 C CNN
-	1    3550 6700
-	0    -1   -1   0
-$EndComp
-Wire Wire Line
-	3400 6600 3900 6600
-Wire Wire Line
-	3900 6700 3750 6700
 Wire Wire Line
 	1700 5100 1800 5100
@@
 NoConn ~ 2700 6900
 NoConn ~ 2700 7000
-Text Label 2700 6600 0    50   ~ 0
-OUT3_P
-Text Label 2700 6700 0    50   ~ 0
-OUT3_N
 NoConn ~ 1300 5700
 NoConn ~ 1300 6200
@@
 P 1200 5150
 F 0 "R10" H 1271 5188 40  0000 L CNN
-F 1 "10K/5%" H 1271 5112 40  0000 L CNN
+F 1 "4.7k/5%" H 1271 5112 40  0000 L CNN
 F 2 "tom-passives:R_0402_1005Metric" V 1130 5150 30  0001 C CNN
 F 3 "" H 1200 5150 30  0000 C CNN
@@
 P 1050 5150
 F 0 "R9" H 1121 5188 40  0000 L CNN
-F 1 "10K/5%" H 1121 5112 40  0000 L CNN
+F 1 "4.7k/5%" H 1121 5112 40  0000 L CNN
 F 2 "tom-passives:R_0402_1005Metric" V 980 5150 30  0001 C CNN
 F 3 "" H 1050 5150 30  0000 C CNN
@@
 Text Label 850  6500 0    50   ~ 0
 XIN
-Wire Wire Line
-	3350 6700 2700 6700
-Wire Wire Line
-	2700 6600 3000 6600
 NoConn ~ 2700 6000
 NoConn ~ 2700 6100
@@
 Text Label 10650 3250 0    50   ~ 0
 CLKIN_N
-$Comp
-L tom-passives:C C?
-U 1 1 5EA5C2D9
-P 3500 5950
-AR Path="/5E98B37D/5EA5C2D9" Ref="C?"  Part="1"
-AR Path="/5EA5C2D9" Ref="C41"  Part="1"
-F 0 "C41" V 3271 5950 40  0000 C CNN
-F 1 "0.1uF/6.3V/X5R/PCIE" V 3347 5950 40  0000 C CNN
-F 2 "tom-passives:C_0402_1005Metric" H 3538 5800 30  0001 C CNN
-F 3 "" H 3500 5950 60  0001 C CNN
-	1    3500 5950
-	-1   0    0    1
-$EndComp
-$Comp
-L tom-passives:C C?
-U 1 1 5EA5CB84
-P 3000 5950
-AR Path="/5E98B37D/5EA5CB84" Ref="C?"  Part="1"
-AR Path="/5EA5CB84" Ref="C40"  Part="1"
-F 0 "C40" V 2771 5950 40  0000 C CNN
-F 1 "0.1uF/6.3V/X5R/PCIE" V 2847 5950 40  0000 C CNN
-F 2 "tom-passives:C_0402_1005Metric" H 3038 5800 30  0001 C CNN
-F 3 "" H 3000 5950 60  0001 C CNN
-	1    3000 5950
-	-1   0    0    1
-$EndComp
-Wire Wire Line
-	3500 6400 3500 6150
-Wire Wire Line
-	3000 6150 3000 6300
 Wire Wire Line
 	3000 6300 2700 6300
-Wire Wire Line
-	3500 5750 3500 5250
-Wire Wire Line
-	3000 5750 3000 5250
 Text Label 3000 5150 1    50   ~ 0
 CLKIN_P
 Text Label 3500 5150 1    50   ~ 0
 CLKIN_N
-Text Label 2700 6300 0    50   ~ 0
-OUT2_P
-Text Label 2700 6400 0    50   ~ 0
-OUT2_N
 Wire Wire Line
 	10600 3450 10650 3450
@@
 P 6400 5200
 F 0 "R51" H 6471 5238 40  0000 L CNN
-F 1 "1K/5%" H 6471 5162 40  0000 L CNN
+F 1 "4.7k/5%" H 6471 5162 40  0000 L CNN
 F 2 "tom-passives:R_0402_1005Metric" V 6330 5200 30  0001 C CNN
 F 3 "" H 6400 5200 30  0000 C CNN
@@
 Wire Wire Line
 	850  5900 600  5900
+Wire Wire Line
+	3000 5250 3000 6300
+Wire Wire Line
+	3500 5250 3500 6400
+Wire Wire Line
+	2700 6600 3900 6600
+Wire Wire Line
+	2700 6700 3900 6700
+$Comp
+L tom-mechanical:TestPoint TP16
+U 1 1 5F400C11
+P 6750 6150
+F 0 "TP16" H 6692 6176 50  0000 R CNN
+F 1 "TestPoint" H 6692 6267 50  0000 R CNN
+F 2 "tom-mechanical:TestPoint_Pad_D1.5mm" H 6950 6150 50  0001 C CNN
+F 3 "~" H 6950 6150 50  0001 C CNN
+	1    6750 6150
+	-1   0    0    1
+$EndComp
+$Comp
+L power:VCC #PWR044
+U 1 1 5F4011B2
+P 6750 6150
+F 0 "#PWR044" H 6750 6000 50  0001 C CNN
+F 1 "VCC" H 6767 6323 50  0000 C CNN
+F 2 "" H 6750 6150 50  0001 C CNN
+F 3 "" H 6750 6150 50  0001 C CNN
+	1    6750 6150
+	1    0    0    -1
+$EndComp
+$Comp
+L tom-mechanical:TestPoint TP18
+U 1 1 5F41DF7B
+P 8250 650
+F 0 "TP18" H 8308 722 50  0000 L CNN
+F 1 "TestPoint" H 8308 677 50  0001 L CNN
+F 2 "tom-mechanical:TestPoint_Pad_D1.5mm" H 8450 650 50  0001 C CNN
+F 3 "~" H 8450 650 50  0001 C CNN
+	1    8250 650
+	1    0    0    -1
+$EndComp
+$Comp
+L tom-mechanical:TestPoint TP19
+U 1 1 5F44DB51
+P 8500 650
+F 0 "TP19" H 8558 722 50  0000 L CNN
+F 1 "TestPoint" H 8558 677 50  0001 L CNN
+F 2 "tom-mechanical:TestPoint_Pad_D1.5mm" H 8700 650 50  0001 C CNN
+F 3 "~" H 8700 650 50  0001 C CNN
+	1    8500 650
+	1    0    0    -1
+$EndComp
+$Comp
+L tom-mechanical:TestPoint TP20
+U 1 1 5F44DEA2
+P 8750 650
+F 0 "TP20" H 8808 722 50  0000 L CNN
+F 1 "TestPoint" H 8808 677 50  0001 L CNN
+F 2 "tom-mechanical:TestPoint_Pad_D1.5mm" H 8950 650 50  0001 C CNN
+F 3 "~" H 8950 650 50  0001 C CNN
+	1    8750 650
+	1    0    0    -1
+$EndComp
+$Comp
+L tom-mechanical:TestPoint TP17
+U 1 1 5F44E186
+P 5700 650
+F 0 "TP17" H 5758 722 50  0000 L CNN
+F 1 "TestPoint" H 5758 677 50  0001 L CNN
+F 2 "tom-mechanical:TestPoint_Pad_D1.5mm" H 5900 650 50  0001 C CNN
+F 3 "~" H 5900 650 50  0001 C CNN
+	1    5700 650
+	1    0    0    -1
+$EndComp
+Wire Wire Line
+	8250 1100 8250 650
+Connection ~ 8250 1100
+Wire Wire Line
+	8500 650  8500 750
+Wire Wire Line
+	8500 750  8350 750
+Wire Wire Line
+	8350 750  8350 1200
+Connection ~ 8350 1200
+Wire Wire Line
+	7900 1400 9350 1400
+Wire Wire Line
+	9350 1300 8450 1300
+Wire Wire Line
+	8350 1200 9350 1200
+Wire Wire Line
+	8250 1100 9350 1100
+Wire Wire Line
+	8750 650  8750 1500
+Connection ~ 8750 1500
+Wire Wire Line
+	8750 1500 8550 1500
+Wire Wire Line
+	5700 650  5700 1800
+Connection ~ 5700 1800
 $EndSCHEMATC

Commit message: v2 hardware: Aug2020/rc2 version - flip tx/rx pairs on s2 - add lcsc part numbers
rc2 errata schematic
- change serial port connector to add +3.3V ? (8-pin)(NO)
- add test points for flash pre-programming
- smaller package on input direction diodes (NO)
- bom dupe errors
- remove all p/s 0R bringup parts
- optimise bom (use 1.5k for led, 10k/4.7k for i2c pullups)
- done led is bright (change to 4.7k)
- improve shield grounding with RC
- check actual values of RGB resistors
- remove caps from clock inputs

rc2 errata pcb
- no gnd marking on serial port connector pins
- change serial port connector to add +3.3V ? (8-pin) (NO)
- no test points for flash pre-programming
- missing caps on xtal? (No but select xtal carefully)
- Cfg sel pins on clock chip?
- No silk on test points
- No +/- pair numbering on silk
- vcc test points for clk pre-programming? (or use bootloader)
- random silk circle under S2
- smaller package on input direction diodes (NO)
- no polarity on 100uF tantalum
- some via in or close to pads
- wrong button package (change from feather to chinese)
- gnd/vcc labels swapped at high end of J2
- clock chip OUT0_SEL_I2CB needs to be tied high after programming
- check teardrops
- power diode footprint marking reverse
- LEDs use cap footprint
Parts:
- added H2, H3, H4: mech-only-no-pins, tom-mechanical:JLCPCB_ASSEMBLY_TOOL_HOLE, symbol tom-mechanical:mech-only-no-pins
- C1: LCSC (none) -> C96123
- C17, C2, C25, C27, C29, C31: LCSC (none) -> C1525
- D1: footprint tom-passives:C_0402_1005Metric -> tom-opto:LED_0402_1005Metric; LCSC (none) -> C130722
- D2: LCSC (none) -> C375571
- D3, D4: symbol tom-passives:DIODE -> tom-semiconductors:DIODE; LCSC (none) -> C146738
- D5: footprint tom-passives:C_0402_1005Metric -> tom-opto:LED_0402_1005Metric; LCSC (none) -> C130724
- H1, J10, J3, J6, J7, J8, SW1, SW2, TP10, TP11, TP12, TP13, TP14, TP15, TP16, TP17, TP18, TP19, TP20, TP9, U1, U2, U4: LCSC (none) -> DNP
- R1, R10, R2, R3, R5, R51, R7, R9: LCSC (none) -> C25900
- R29, R37: LCSC (none) -> C25867
- R30, R4: LCSC (none) -> C11702
- R34, R35: LCSC (none) -> C25099
- R52: LCSC (none) -> C25076
- R6: LCSC (none) -> C25882
- X1: LCSC (none) -> C9006
Connections:
- net VBUS: now also D4.2 (A); no longer D4.1 (A)
- net VCC: now also D3.1 (K), D4.1 (K); no longer D3.2 (K), D4.2 (K)
- net VCC_IN: now also D3.2 (A); no longer D3.1 (A)

Commit message: JLC power supplies almost routed VCCBRAM to go Need to - check BOM - add power good leds - fix vccbram inc caps - fix 100uF part number - update silk
Parts:
- removed J3: JTAG_EN, tom-connectors:PinHeader_1x02_P1.27mm_Vertical, symbol tom-connectors:Conn_01x02
- removed R4: 1k/1%, tom-passives:R_0402_1005Metric, symbol tom-passives:R
Connections:
- net M2 is gone; now on net GND: U1.U9 (M2_0)
Changed lines of the file:
@@
-$EndComp
-$Comp
-L tom-passives:R R4
-U 1 1 5E7FB45A
-P 5850 2450
-F 0 "R4" H 5921 2488 40  0000 L CNN
-F 1 "1k/1%" H 5921 2412 40  0000 L CNN
-F 2 "tom-passives:R_0402_1005Metric" V 5780 2450 30  0001 C CNN
-F 3 "" H 5850 2450 30  0000 C CNN
-F 4 "C11702" H 5850 2450 50  0001 C CNN "LCSC"
-	1    5850 2450
-	1    0    0    -1
-$EndComp
-$Comp
-L power:GND #PWR013
-U 1 1 5E7FCD8A
-P 5850 2700
-F 0 "#PWR013" H 5850 2450 50  0001 C CNN
-F 1 "GND" H 5855 2527 50  0000 C CNN
-F 2 "" H 5850 2700 50  0001 C CNN
-F 3 "" H 5850 2700 50  0001 C CNN
-	1    5850 2700
-	1    0    0    -1
 $EndComp
 $Comp
@@
 	8450 2000 6150 2000
 $Comp
-L tom-connectors:Conn_01x02 J3
-U 1 1 5E81BC64
-P 6350 2550
-F 0 "J3" V 6222 2630 50  0000 L CNN
-F 1 "JTAG_EN" V 6313 2630 50  0000 L CNN
-F 2 "tom-connectors:PinHeader_1x02_P1.27mm_Vertical" H 6350 2550 50  0001 C CNN
-F 3 "~" H 6350 2550 50  0001 C CNN
-F 4 "DNP" H 6350 2550 50  0001 C CNN "LCSC"
-	1    6350 2550
-	0    1    1    0
-$EndComp
-Wire Wire Line
-	5850 2200 6250 2200
-Wire Wire Line
-	6250 2200 6250 2350
-Connection ~ 5850 2200
-$Comp
-L power:+3V3 #PWR016
-U 1 1 5E82C135
-P 6350 2350
-F 0 "#PWR016" H 6350 2200 50  0001 C CNN
-F 1 "+3V3" H 6365 2523 50  0000 C CNN
-F 2 "" H 6350 2350 50  0001 C CNN
-F 3 "" H 6350 2350 50  0001 C CNN
-	1    6350 2350
-	1    0    0    -1
-$EndComp
-$Comp
 L tom-mechanical:SW_SPST SW1
 U 1 1 5E83A5C8
@@
 	1    0    0    -1
 $EndComp
-Text Label 5350 2200 0    50   ~ 0
+Text Label 3550 2200 0    50   ~ 0
 M2
-Wire Wire Line
-	3450 2200 5850 2200
 $Comp
 L power:+3V3 #PWR01
@@
 	1    0    0    -1
 $EndComp
+Wire Wire Line
+	3450 2200 4850 2200
+Wire Wire Line
+	4850 2100 4850 2200
+Connection ~ 4850 2100
 $EndSCHEMATC

Commit message: v2 hardware updates: fixed inductor footprint, updates for DFA
Parts:
- H2, H3, H4: LCSC (none) -> DNP
- R30: value 1k/1% -> 1.2k/1%; LCSC C11702 -> C25862
- R34, R35: value 270R/5% -> 300R/5%; LCSC C25099 -> C25102
Changed lines of the file:
@@
 P 8950 2500
 F 0 "R30" V 8765 2500 40  0000 C CNN
-F 1 "1k/1%" V 8841 2500 40  0000 C CNN
+F 1 "1.2k/1%" V 8841 2500 40  0000 C CNN
 F 2 "tom-passives:R_0402_1005Metric" V 8880 2500 30  0001 C CNN
 F 3 "" H 8950 2500 30  0000 C CNN
-F 4 "C11702" H 8950 2500 50  0001 C CNN "LCSC"
+F 4 "C25862" H 8950 2500 50  0001 C CNN "LCSC"
 	1    8950 2500
 	0    1    1    0
@@
 P 8950 2700
 F 0 "R34" V 8850 2700 40  0000 C CNN
-F 1 "270R/5%" V 9050 2700 40  0000 C CNN
+F 1 "300R/5%" V 9050 2700 40  0000 C CNN
 F 2 "tom-passives:R_0402_1005Metric" V 8880 2700 30  0001 C CNN
 F 3 "" H 8950 2700 30  0000 C CNN
-F 4 "C25099" H 8950 2700 50  0001 C CNN "LCSC"
+F 4 "C25102" H 8950 2700 50  0001 C CNN "LCSC"
 	1    8950 2700
 	0    1    1    0
@@
 P 8950 2900
 F 0 "R35" V 9050 2900 40  0000 C CNN
-F 1 "270R/5%" V 9150 2900 40  0000 C CNN
+F 1 "300R/5%" V 9150 2900 40  0000 C CNN
 F 2 "tom-passives:R_0402_1005Metric" V 8880 2900 30  0001 C CNN
 F 3 "" H 8950 2900 30  0000 C CNN
-F 4 "C25099" H 8950 2900 50  0001 C CNN "LCSC"
+F 4 "C25102" H 8950 2900 50  0001 C CNN "LCSC"
 	1    8950 2900
 	0    1    1    0
@@
 F 2 "tom-mechanical:JLCPCB_ASSEMBLY_TOOL_HOLE" H 9050 6650 50  0001 C CNN
 F 3 "" H 9050 6650 50  0001 C CNN
+F 4 "DNP" H 9050 6650 50  0001 C CNN "LCSC"
 	1    9050 6650
 	1    0    0    -1
@@
 F 2 "tom-mechanical:JLCPCB_ASSEMBLY_TOOL_HOLE" H 9050 6850 50  0001 C CNN
 F 3 "" H 9050 6850 50  0001 C CNN
+F 4 "DNP" H 9050 6850 50  0001 C CNN "LCSC"
 	1    9050 6850
 	1    0    0    -1
@@
 F 2 "tom-mechanical:JLCPCB_ASSEMBLY_TOOL_HOLE" H 9050 7050 50  0001 C CNN
 F 3 "" H 9050 7050 50  0001 C CNN
+F 4 "DNP" H 9050 7050 50  0001 C CNN "LCSC"
 	1    9050 7050
 	1    0    0    -1

Commit message: hardware: minor fixes to v2 for Nov2020 run
Parts:
- added D6: PWR, tom-opto:LED_0402_1005Metric, symbol tom-opto:LED
- added R4: 4.7k/5%, tom-passives:R_0402_1005Metric, symbol tom-passives:R
Connections:
- net +3V3: now also R4.1
- net GND: now also D6.1 (K)
- new net: D6.2 (A), R4.2
Changed lines of the file:
@@
 	4850 2100 4850 2200
 Connection ~ 4850 2100
+$Comp
+L tom-opto:LED D6
+U 1 1 5FDAD48B
+P 6000 5600
+F 0 "D6" V 6039 5483 50  0000 R CNN
+F 1 "PWR" V 5948 5483 50  0000 R CNN
+F 2 "tom-opto:LED_0402_1005Metric" H 6000 5600 50  0001 C CNN
+F 3 "~" H 6000 5600 50  0001 C CNN
+F 4 "C130724" H 6000 5600 50  0001 C CNN "LCSC"
+	1    6000 5600
+	0    -1   -1   0
+$EndComp
+$Comp
+L tom-passives:R R4
+U 1 1 5FDAD8DC
+P 6000 5200
+F 0 "R4" H 6071 5238 40  0000 L CNN
+F 1 "4.7k/5%" H 6071 5162 40  0000 L CNN
+F 2 "tom-passives:R_0402_1005Metric" V 5930 5200 30  0001 C CNN
+F 3 "" H 6000 5200 30  0000 C CNN
+F 4 "C25900" H 6000 5200 50  0001 C CNN "LCSC"
+	1    6000 5200
+	1    0    0    -1
+$EndComp
+$Comp
+L power:+3V3 #PWR0170
+U 1 1 5FDAD8E6
+P 6000 4950
+F 0 "#PWR0170" H 6000 4800 50  0001 C CNN
+F 1 "+3V3" H 6015 5123 50  0000 C CNN
+F 2 "" H 6000 4950 50  0001 C CNN
+F 3 "" H 6000 4950 50  0001 C CNN
+	1    6000 4950
+	1    0    0    -1
+$EndComp
+$Comp
+L power:GND #PWR0171
+U 1 1 5FDAD8F0
+P 6000 5750
+F 0 "#PWR0171" H 6000 5500 50  0001 C CNN
+F 1 "GND" H 6005 5577 50  0000 C CNN
+F 2 "" H 6000 5750 50  0001 C CNN
+F 3 "" H 6000 5750 50  0001 C CNN
+	1    6000 5750
+	1    0    0    -1
+$EndComp
 $EndSCHEMATC
